Commit message: hardware interface base + gazebo ignition + organizing + fixes

File: description/gazebo_ros2_control.xacro (robot description, xacro)
@@ -3,5 +3,5 @@
     <ros2_control name="GazeboSystem" type="system">
         <hardware>
-            <plugin>gazebo_ros2_control/GazeboSystem</plugin>
+            <plugin>gz_ros2_control/GazeboSimSystem</plugin>
         </hardware>
          <joint name="wheel_front_left_joint">
@@ -9,5 +9,4 @@
             <state_interface name="position"/>
             <state_interface name="velocity"/>
-            <state_interface name="effort"/>
         </joint>
         <joint name="wheel_front_right_joint">
@@ -15,5 +14,4 @@
             <state_interface name="position"/>
             <state_interface name="velocity"/>
-            <state_interface name="effort"/>
         </joint>
         <joint name="wheel_rear_left_joint">
@@ -21,5 +19,4 @@
             <state_interface name="position"/>
             <state_interface name="velocity"/>
-            <state_interface name="effort"/>
         </joint>
         <joint name="wheel_rear_right_joint">
@@ -27,25 +24,10 @@
             <state_interface name="position"/>
             <state_interface name="velocity"/>
-            <state_interface name="effort"/>
         </joint>
-        <!--
-        <joint name="wheel_left_joint">
-            <command_interface name="velocity"/>
-            <state_interface name="position"/>
-            <state_interface name="velocity"/>
-            <state_interface name="effort"/>
-        </joint>
-        <joint name="wheel_right_joint">
-            <command_interface name="velocity"/>
-            <state_interface name="position"/>
-            <state_interface name="velocity"/>
-            <state_interface name="effort"/>
-        </joint>
-        -->
     </ros2_control>
-    <!-- ROS 2 Control plugin for Gazebo -->
     <gazebo>
-        <plugin name="gazebo_ros2_control" filename="libgazebo_ros2_control.so">
-            <parameters>$(find usb_ros2_state)/config/parameter.yaml</parameters>
+        <plugin name="gz_ros2_control::GazeboSimROS2ControlPlugin" filename="libgz_ros2_control-system.so">
+            <parameters>$(find quac)/config/controllers.yaml</parameters>
+            <parameters>$(find quac)/config/gz_sim_time.yaml</parameters>
         </plugin>
     </gazebo>

File: description/lidar.xacro (robot description, xacro)
@@ -36,9 +36,9 @@
     <gazebo reference="laser_frame">
         <material>Gazebo/Red</material>
-        <sensor name="laser" type="ray">
+        <sensor name="laser" type="gpu_lidar">
             <pose> 0 0 0 0 0 0 </pose>
-            <visualize>true</visualize>
+            <visualize>false</visualize>
             <update_rate>10</update_rate>
-            <ray>
+            <lidar>
                 <scan>
                     <horizontal>
@@ -52,12 +52,7 @@
                     <max>12</max>
                 </range>
-            </ray>
-            <plugin name="laser_controller" filename="libgazebo_ros_ray_sensor.so">
-                <ros>
-                    <argument>~/out:=scan</argument>
-                </ros>
-                <output_type>sensor_msgs/LaserScan</output_type>
-                <frame_name>laser_frame</frame_name>
-            </plugin>
+            </lidar>
+            <topic>scan</topic>
+            <gz_frame_id>laser_frame</gz_frame_id>
         </sensor>
     </gazebo>

File: description/robot.urdf.xacro (robot description, xacro)
@@ -1,7 +1,12 @@
 <?xml version="1.0"?>
-<robot xmlns:xacro="http://www.ros.org/wiki/xacro"  name="robot">
+<robot xmlns:xacro="http://www.ros.org/wiki/xacro"  name="quac_robot">
     <xacro:include filename="robot_core.xacro" />
     <xacro:include filename="lidar.xacro" />
-    <!-- -->
-    <xacro:include filename="ddsm_control.xacro" />
+    <xacro:arg name="sim_mode" default="false"/>
+    <xacro:if value="$(arg sim_mode)">
+        <xacro:include filename="gazebo_ros2_control.xacro" />
+    </xacro:if>
+    <xacro:unless value="$(arg sim_mode)">
+        <xacro:include filename="ros2_control.xacro" />
+    </xacro:unless>
 </robot>

File: description/robot_core.xacro (robot description, xacro)
@@ -38,5 +38,5 @@
             <origin xyz="0 0 0" rpy="0 0 0"/>
             <geometry>
-            <mesh filename="package://usb_ros2_state/meshes/base_link.stl" scale="${mesh_scale} ${mesh_scale} ${mesh_scale}"/>
+            <mesh filename="package://quac/meshes/base_link.stl" scale="${mesh_scale} ${mesh_scale} ${mesh_scale}"/>
             </geometry>
             <material name="chassis_material"/>
@@ -45,5 +45,5 @@
             <origin xyz="0 0 0" rpy="0 0 0"/>
             <geometry>
-            <mesh filename="package://usb_ros2_state/meshes/base_link.stl" scale="${mesh_scale} ${mesh_scale} ${mesh_scale}"/>
+            <mesh filename="package://quac/meshes/base_link.stl" scale="${mesh_scale} ${mesh_scale} ${mesh_scale}"/>
             </geometry>
         </collision>
@@ -55,66 +55,4 @@
         <gravity>true</gravity>
     </gazebo>
-    <xacro:macro name="wheel_visual" params="name joint_origin_xyz">
-        <joint name="${name}_joint" type="fixed">
-            <origin xyz="${joint_origin_xyz}" rpy="0 0 0"/>
-            <parent link="chassis"/>
-            <child link="${name}"/>
-            <axis xyz="-1.0 0.0 0.0"/>
-        </joint>
-        <link name="${name}">
-            <inertial>
-                <origin xyz="0 0 0" rpy="0 0 0"/>
-                <mass value="1.0"/>
-                <inertia ixx="0.0" iyy="0.0" izz="0.0" ixy="0.0" iyz="0.0" ixz="0.0"/>
-            </inertial>
-            <visual>
-                <origin xyz="0 0 0" rpy="0 ${-pi/2} 0"/>
-                <geometry>
-                    <cylinder radius="0.05" length="0.04"/>
-                </geometry>
-                <material name="wheel_material"/>
-            </visual>
-            <collision>
-                <origin xyz="0 0 0" rpy="0 ${-pi/2} 0"/>
-                <geometry>
-                    <cylinder radius="0.05" length="0.04"/>
-                </geometry>
-            </collision>
-        </link>
-        <gazebo reference="${name}">
-            <material>Gazebo/Black</material>
-            <mu1 value="0.001"/>
-            <mu2 value="0.001"/>
-        </gazebo>
-    </xacro:macro>
-    <xacro:macro name="wheel_real" params="name joint_origin_xyz">
-        <joint name="${name}_joint" type="continuous">
-            <origin xyz="${joint_origin_xyz}" rpy="0 0 0"/>
-            <parent link="chassis"/>
-            <child link="${name}"/>
-            <axis xyz="-1.0 0.0 0.0"/>
-        </joint>
-        <link name="${name}">
-            <xacro:inertial_cylinder mass="0.1" length="0.04" radius="0.05">
-                <origin xyz="0 0 0" rpy="0 ${-pi/2} 0"/>
-            </xacro:inertial_cylinder>
-            <collision>
-                <origin xyz="0 0 0" rpy="0 ${-pi/2} 0"/>
-                <geometry>
-                    <cylinder radius="0.05" length="0.04"/>
-                </geometry>
-            </collision>
-        </link>
-        <transmission name="${name}_trans">
-            <type>transmission_interface/SimpleTransmission</type>
-            <joint name="${name}_joint">
-                <hardware_interface>velocity</hardware_interface>
-            </joint>
-            <actuator name="${name}_motor">
-                <hardware_interface>velocity</hardware_interface>
-                <mechanicalReduction>1</mechanicalReduction>
-            </actuator>
-        </transmission>
-    </xacro:macro>
     <xacro:macro name="wheel" params="name joint_origin_xyz link_xyz mesh">
         <joint name="${name}_joint" type="continuous">
@@ -163,5 +101,5 @@
         joint_origin_xyz="0.105 -0.104 -0.0183"
         link_xyz="-0.105 0.104 0.0183"
-        mesh="package://usb_ros2_state/meshes/wheel.stl"
+        mesh="package://quac/meshes/wheel.stl"
         />
     <xacro:wheel
@@ -169,5 +107,5 @@
         joint_origin_xyz="0.105 0.104 -0.0183"
         link_xyz="-0.105 -0.104 0.0183"
-        mesh="package://usb_ros2_state/meshes/wheel_2.stl"
+        mesh="package://quac/meshes/wheel_2.stl"
         />
     <xacro:wheel
@@ -175,5 +113,5 @@
         joint_origin_xyz="-0.105 0.104 -0.0183"
         link_xyz="0.105 -0.104 0.0183"
-        mesh="package://usb_ros2_state/meshes/wheel_3.stl"
+        mesh="package://quac/meshes/wheel_3.stl"
         />
     <xacro:wheel
@@ -181,31 +119,5 @@
         joint_origin_xyz="-0.105 -0.104 -0.0183"
         link_xyz="0.105 0.104 0.0183"
-        mesh="package://usb_ros2_state/meshes/wheel_4.stl"
+        mesh="package://quac/meshes/wheel_4.stl"
         />
-    <!--
-    <xacro:wheel_visual
-        name="wheel_rear_right"
-        joint_origin_xyz="0.105 -0.104 -0.0183"
-        />
-    <xacro:wheel_visual
-        name="wheel_front_right"
-        joint_origin_xyz="0.105 0.104 -0.0183"
-        />
-    <xacro:wheel_visual
-        name="wheel_front_left"
-        joint_origin_xyz="-0.105 0.104 -0.0183"
-        />
-    <xacro:wheel_visual
-        name="wheel_rear_left"
-        joint_origin_xyz="-0.105 -0.104 -0.0183"
-        />
-    <xacro:wheel_real
-        name="wheel_left"
-        joint_origin_xyz="-0.105 0.0 -0.0183"
-        />
-    <xacro:wheel_real
-        name="wheel_right"
-        joint_origin_xyz="0.105 0.0 -0.0183"
-        />
-    -->
 </robot>

File: description/ros2_control.xacro (robot description, xacro)
@@ -1,7 +1,7 @@
 <?xml version="1.0"?>
 <robot xmlns:xacro="http://www.ros.org/wiki/xacro">
-    <ros2_control name="MyRobotHW" type="system">
+    <ros2_control name="quac_hardware" type="system">
     <hardware>
-        <plugin>quac_hardware/DDSMHardware</plugin>
+        <plugin>quac_hardware/DiffDriveDDSM115</plugin>
     </hardware>
     <joint name="wheel_front_left_joint">
@@ -9,5 +9,5 @@
         <state_interface name="position"/>
         <state_interface name="velocity"/>
-        <state_interface name="effort"/>
+        <param name="id">1</param>
     </joint>
     <joint name="wheel_front_right_joint">
@@ -15,5 +15,5 @@
         <state_interface name="position"/>
         <state_interface name="velocity"/>
-        <state_interface name="effort"/>
+        <param name="id">2</param>
     </joint>
     <joint name="wheel_rear_left_joint">
@@ -21,5 +21,5 @@
         <state_interface name="position"/>
         <state_interface name="velocity"/>
-        <state_interface name="effort"/>
+        <param name="id">3</param>
     </joint>
     <joint name="wheel_rear_right_joint">
@@ -27,5 +27,5 @@
         <state_interface name="position"/>
         <state_interface name="velocity"/>
-        <state_interface name="effort"/>
+        <param name="id">4</param>
     </joint>
 </ros2_control>
