Commit message: hardware adaption

File: description/lidar.xacro (robot description, xacro)
@@ -16,5 +16,5 @@
         <parent link="chassis"/>
         <child link="laser_frame"/>
-        <origin xyz="0.0 0.1 0.04" rpy="0 0 ${pi/2}"/>
+        <origin xyz="0.0 -0.104 0.04" rpy="0 0 3.6"/>
     </joint>
     <link name="laser_frame">

File: description/ros2_control.xacro (robot description, xacro)
@@ -4,5 +4,5 @@
     <hardware>
         <plugin>quac_hardware/DiffDriveDDSM115</plugin>
-        <param name="port">/dev/ttyAMA0</param>
+        <param name="port">/dev/ttyACM0</param>
         <param name="encoder_resolution">4096</param>
         <param name="act">6</param>

Commit message: hardware adaptaion

File: description/lidar.xacro (robot description, xacro)
@@ -16,5 +16,5 @@
         <parent link="chassis"/>
         <child link="laser_frame"/>
-        <origin xyz="0.0 -0.104 0.04" rpy="0 0 3.6"/>
+        <origin xyz="0.0 -0.03 0.04" rpy="0 0 ${-pi/2}"/>
     </joint>
     <link name="laser_frame">

File: description/ros2_control.xacro (robot description, xacro)
@@ -4,8 +4,23 @@
     <hardware>
         <plugin>quac_hardware/DiffDriveDDSM115</plugin>
-        <param name="port">/dev/ttyUSB0</param>
+        <param name="port">/dev/ttyUSB1</param>
         <param name="act">1</param>
+        <param name="feedback">true</param>
     </hardware>
     <joint name="wheel_front_left_joint">
+        <command_interface name="velocity"/>
+        <state_interface name="position"/>
+        <state_interface name="velocity"/>
+        <param name="id">4</param>
+        <param name="scalar">1</param>
+    </joint>
+    <joint name="wheel_front_right_joint">
+        <command_interface name="velocity"/>
+        <state_interface name="position"/>
+        <state_interface name="velocity"/>
+        <param name="id">1</param>
+        <param name="scalar">-1</param>
+    </joint>
+    <joint name="wheel_rear_left_joint">
         <command_interface name="velocity"/>
         <state_interface name="position"/>
@@ -14,23 +29,9 @@
         <param name="scalar">1</param>
     </joint>
-    <joint name="wheel_front_right_joint">
-        <command_interface name="velocity"/>
-        <state_interface name="position"/>
-        <state_interface name="velocity"/>
-        <param name="id">4</param>
-        <param name="scalar">-1</param>
-    </joint>
-    <joint name="wheel_rear_left_joint">
+    <joint name="wheel_rear_right_joint">
         <command_interface name="velocity"/>
         <state_interface name="position"/>
         <state_interface name="velocity"/>
         <param name="id">2</param>
-        <param name="scalar">1</param>
-    </joint>
-    <joint name="wheel_rear_right_joint">
-        <command_interface name="velocity"/>
-        <state_interface name="position"/>
-        <state_interface name="velocity"/>
-        <param name="id">1</param>
         <param name="scalar">-1</param>
     </joint>
