Commit message: refactoring + arm

File: description/robot.urdf.xacro (robot description, xacro)
@@ -1,9 +1,8 @@
 <?xml version="1.0"?>
 <robot xmlns:xacro="http://www.ros.org/wiki/xacro"  name="quac_robot">
-    <xacro:include filename="robot_core.xacro" />
-    <xacro:include filename="lidar.xacro" />
+    <xacro:include filename="urdf/robot_core.xacro" />
     <xacro:arg name="sim_mode" default="false"/>
     <xacro:if value="$(arg sim_mode)">
-        <xacro:include filename="gazebo_ros2_control.xacro" />
+        <xacro:include filename="gazebo.xacro" />
     </xacro:if>
     <xacro:unless value="$(arg sim_mode)">

File: description/ros2_control.xacro (robot description, xacro)
@@ -2,38 +2,38 @@
 <robot xmlns:xacro="http://www.ros.org/wiki/xacro">
     <ros2_control name="quac_hardware" type="system">
-    <hardware>
-        <plugin>quac_hardware/DiffDriveDDSM115</plugin>
-        <param name="port">/dev/ttyUSB1</param>
-        <param name="act">1</param>
-        <param name="feedback">true</param>
-    </hardware>
-    <joint name="wheel_front_left_joint">
-        <command_interface name="velocity"/>
-        <state_interface name="position"/>
-        <state_interface name="velocity"/>
-        <param name="id">4</param>
-        <param name="scalar">1</param>
-    </joint>
-    <joint name="wheel_front_right_joint">
-        <command_interface name="velocity"/>
-        <state_interface name="position"/>
-        <state_interface name="velocity"/>
-        <param name="id">1</param>
-        <param name="scalar">-1</param>
-    </joint>
-    <joint name="wheel_rear_left_joint">
-        <command_interface name="velocity"/>
-        <state_interface name="position"/>
-        <state_interface name="velocity"/>
-        <param name="id">3</param>
-        <param name="scalar">1</param>
-    </joint>
-    <joint name="wheel_rear_right_joint">
-        <command_interface name="velocity"/>
-        <state_interface name="position"/>
-        <state_interface name="velocity"/>
-        <param name="id">2</param>
-        <param name="scalar">-1</param>
-    </joint>
-</ros2_control>
+        <hardware>
+            <plugin>quac_hardware/DDSM115</plugin>
+            <param name="port">/dev/ttyUSB1</param>
+            <param name="act">1</param>
+            <param name="feedback">true</param>
+        </hardware>
+        <joint name="wheel_front_left_joint">
+            <command_interface name="velocity"/>
+            <state_interface name="position"/>
+            <state_interface name="velocity"/>
+            <param name="id">4</param>
+            <param name="scalar">1</param>
+        </joint>
+        <joint name="wheel_front_right_joint">
+            <command_interface name="velocity"/>
+            <state_interface name="position"/>
+            <state_interface name="velocity"/>
+            <param name="id">1</param>
+            <param name="scalar">-1</param>
+        </joint>
+        <joint name="wheel_rear_left_joint">
+            <command_interface name="velocity"/>
+            <state_interface name="position"/>
+            <state_interface name="velocity"/>
+            <param name="id">3</param>
+            <param name="scalar">1</param>
+        </joint>
+        <joint name="wheel_rear_right_joint">
+            <command_interface name="velocity"/>
+            <state_interface name="position"/>
+            <state_interface name="velocity"/>
+            <param name="id">2</param>
+            <param name="scalar">-1</param>
+        </joint>
+    </ros2_control>
 </robot>

File: description/urdf/lidar.xacro (robot description, xacro)
@@ -15,8 +15,8 @@
     <joint name="lidar_joint" type="fixed">
         <parent link="chassis"/>
-        <child link="laser_frame"/>
+        <child link="lidar"/>
         <origin xyz="0.0 -0.03 0.04" rpy="0 0 ${-pi/2}"/>
     </joint>
-    <link name="laser_frame">
+    <link name="lidar">
         <visual>
             <geometry>
@@ -34,26 +34,3 @@
         </xacro:inertial_cylinder>
     </link>
-    <gazebo reference="laser_frame">
-        <material>Gazebo/Red</material>
-        <sensor name="laser" type="gpu_lidar">
-            <pose> 0 0 0 0 0 0 </pose>
-            <visualize>false</visualize>
-            <update_rate>10</update_rate>
-            <lidar>
-                <scan>
-                    <horizontal>
-                        <samples>360</samples>
-                        <min_angle>-3.14</min_angle>
-                        <max_angle>3.14</max_angle>
-                    </horizontal>
-                </scan>
-                <range>
-                    <min>0.3</min>
-                    <max>12</max>
-                </range>
-            </lidar>
-            <topic>scan</topic>
-            <gz_frame_id>laser_frame</gz_frame_id>
-        </sensor>
-    </gazebo>
 </robot>

File: description/urdf/wheels.xacro (robot description, xacro)
@@ -1,58 +1,5 @@
 <?xml version="1.0"?>
 <robot xmlns:xacro="http://www.ros.org/wiki/xacro">
-    <xacro:macro name="inertial_cylinder" params="mass length radius *origin">
-        <inertial>
-            <xacro:insert_block name="origin"/>
-            <mass value="${mass}" />
-            <inertia ixx="${(1/12) * mass * (3*radius*radius + length*length)}" ixy="0.0" ixz="0.0"
-                    iyy="${(1/12) * mass * (3*radius*radius + length*length)}" iyz="0.0"
-                    izz="${(1/2) * mass * (radius*radius)}" />
-        </inertial>
-    </xacro:macro>
     <xacro:property name="mesh_scale" value="0.001"/>
-    <material name="chassis_material">
-        <color rgba="1.0 1.0 1.0 1.0" />
-    </material>
-    <material name="wheel_material">
-        <color rgba="0.6 0.6 0.6 1.0" />
-    </material>
-    <link name="base_link"/>
-    <joint name="base_footprint_joint" type="fixed">
-        <parent link="base_link"/>
-        <child link="base_footprint"/>
-        <origin xyz="0 0 0" rpy="0 0 0"/>
-    </joint>
-    <link name="base_footprint"/>
-    <joint name="chassis_joint" type="fixed">
-        <parent link="base_link"/>
-        <child link="chassis"/>
-        <origin xyz="0 0 0.0" rpy="0 0 ${-pi/2}"/>
-    </joint>
-    <link name="chassis">
-        <inertial>
-            <origin xyz="-7.066717348492194e-05 3.485618129802738e-05 0.00889428874586655" rpy="0 0 0"/>
-            <mass value="2.985747783671821"/>
-            <inertia ixx="0.025172" iyy="0.005971" izz="0.030362" ixy="-6e-06" iyz="2e-06" ixz="-2e-06"/>
-        </inertial>
-        <visual>
-            <origin xyz="0 0 0" rpy="0 0 0"/>
-            <geometry>
-            <mesh filename="package://quac/meshes/base_link.stl" scale="${mesh_scale} ${mesh_scale} ${mesh_scale}"/>
-            </geometry>
-            <material name="chassis_material"/>
-        </visual>
-        <collision>
-            <origin xyz="0 0 0" rpy="0 0 0"/>
-            <geometry>
-            <mesh filename="package://quac/meshes/base_link.stl" scale="${mesh_scale} ${mesh_scale} ${mesh_scale}"/>
-            </geometry>
-        </collision>
-    </link>
-    <gazebo reference="chassis">
-        <material>Gazebo/White</material>
-        <mu1>0.2</mu1>
-        <mu2>0.2</mu2>
-        <gravity>true</gravity>
-    </gazebo>
     <xacro:macro name="wheel" params="name joint_origin_xyz link_xyz mesh">
         <joint name="${name}_joint" type="continuous">
@@ -90,14 +37,4 @@
             </gazebo>
         </link>
-        <transmission name="${name}_trans">
-            <type>transmission_interface/SimpleTransmission</type>
-            <joint name="${name}_joint">
-                <hardware_interface>velocity</hardware_interface>
-            </joint>
-            <actuator name="${name}_motor">
-                <hardware_interface>velocity</hardware_interface>
-                <mechanicalReduction>1</mechanicalReduction>
-            </actuator>
-        </transmission>
         <gazebo reference="${name}">
             <material>Gazebo/Black</material>

Commit message: new robot model

File: description/robot.urdf.xacro (robot description, xacro)
@@ -5,5 +5,4 @@
     <xacro:include filename="urdf/servo.xacro" />
     <xacro:include filename="urdf/chassis.xacro" />
-    <xacro:include filename="urdf/lidar.xacro" />
     <xacro:include filename="urdf/wheels.xacro" />
     <xacro:include filename="urdf/arm.xacro" />

File: description/urdf/arm.xacro (robot description, xacro)
@@ -12,12 +12,4 @@
                 <material name="orange" />
             </visual>
-            <collision>
-                <geometry>
-                    <box size="${plate_x} ${plate_y} ${plate_z}" />
-                </geometry>
-            </collision>
-            <xacro:inertial_box mass="0.1" x="${plate_x}" y="${plate_y}" z="${plate_z}">
-                <origin xyz="0 0 0" rpy="0 0 0"/>
-            </xacro:inertial_box>
         </link>
     </xacro:macro>
@@ -39,5 +31,5 @@
         <parent link="chassis" />
         <child link="arm_servo_0_axis" />
-        <origin xyz="0.0 0.135 0.04" rpy="0 ${pi/2} 0" />
+        <origin xyz="0.135 0.0 0.04" rpy="${pi/2} ${pi/2} 0" />
     </joint>
     <xacro:servo_flipped name="arm_servo_0"/>
@@ -95,5 +87,5 @@
             </geometry>
         </collision>
-        <xacro:inertial_cylinder mass="0.1" length="0.04" radius="0.02">
+        <xacro:inertial_cylinder mass="0.1" length="0.02" radius="0.02">
             <origin xyz="0 0 0" rpy="0 0 0"/>
         </xacro:inertial_cylinder>

File: description/urdf/chassis.xacro (robot description, xacro)
@@ -10,16 +10,16 @@
         <parent link="base_link"/>
         <child link="chassis"/>
-        <origin xyz="0 0 0.07" rpy="0 0 ${-pi/2}"/>
+        <origin xyz="0 0 0.09705" rpy="0 0 0"/>
     </joint>
     <link name="chassis">
         <inertial>
-            <origin xyz="-7.066717348492194e-05 3.485618129802738e-05 0.00889428874586655" rpy="0 0 0"/>
-            <mass value="2.985747783671821"/>
-            <inertia ixx="0.025172" iyy="0.005971" izz="0.030362" ixy="-6e-06" iyz="2e-06" ixz="-2e-06"/>
+            <origin xyz="-0.006592503505638408 -1.5301626995551604e-17 0.04294027543409115" rpy="0 0 0"/>
+            <mass value="6.419279977222798"/>
+            <inertia ixx="0.031932" iyy="0.058111" izz="0.057234" ixy="-0.0" iyz="-0.0" ixz="0.003075"/>
         </inertial>
         <visual>
             <origin xyz="0 0 0" rpy="0 0 0"/>
             <geometry>
-                <mesh filename="package://quac/meshes/base_link.stl" scale="${mesh_scale} ${mesh_scale} ${mesh_scale}"/>
+                <mesh filename="package://quac/meshes/chassis.stl" scale="${mesh_scale} ${mesh_scale} ${mesh_scale}"/>
             </geometry>
             <material name="chassis_material"/>
@@ -28,5 +28,5 @@
             <origin xyz="0 0 0" rpy="0 0 0"/>
             <geometry>
-                <mesh filename="package://quac/meshes/base_link.stl" scale="${mesh_scale} ${mesh_scale} ${mesh_scale}"/>
+                <mesh filename="package://quac/meshes/chassis.stl" scale="${mesh_scale} ${mesh_scale} ${mesh_scale}"/>
             </geometry>
         </collision>
@@ -38,3 +38,12 @@
         <gravity>true</gravity>
     </gazebo>
+    <material name="lidar_material">
+        <color rgba="0.8 0.2 0.2 1.0" />
+    </material>
+    <joint name="lidar_joint" type="fixed">
+        <parent link="chassis"/>
+        <child link="lidar"/>
+        <origin xyz="-0.02 0.0 0.15" rpy="0 0 0"/>
+    </joint>
+    <link name="lidar"/>
 </robot>

File: description/urdf/wheels.xacro (robot description, xacro)
@@ -1,30 +1,28 @@
 <?xml version="1.0"?>
 <robot xmlns:xacro="http://www.ros.org/wiki/xacro">
-    <xacro:macro name="wheel" params="name joint_origin_xyz link_xyz mesh">
+    <xacro:macro name="wheel" params="name xyz">
         <joint name="${name}_joint" type="continuous">
-            <origin xyz="${joint_origin_xyz}" rpy="0 0 0"/>
+            <origin xyz="${xyz}" rpy="0 0 0"/>
             <parent link="chassis"/>
             <child link="${name}"/>
-            <axis xyz="-1.0 0.0 0.0"/>
+            <axis xyz="0.0 1.0 0.0"/>
         </joint>
         <link name="${name}">
-            <inertial>
-                <origin xyz="0 0 0" rpy="0 0 0"/>
-                <mass value="1.0708903957924194"/>
-                <inertia ixx="0.001339" iyy="0.000897" izz="0.000897" ixy="0.0" iyz="0.0" ixz="0.0"/>
-            </inertial>
             <visual>
-                <origin xyz="${link_xyz}" rpy="0 0 0"/>
+                <origin xyz="0 0 0" rpy="${pi/2} 0 0"/>
                 <geometry>
-                    <mesh filename="${mesh}" scale="${mesh_scale} ${mesh_scale} ${mesh_scale}"/>
+                    <cylinder radius="0.06" length="0.04" />
                 </geometry>
-                <material name="wheel_material"/>
+                <material name="black" />
             </visual>
             <collision>
-                <origin xyz="${link_xyz}" rpy="0 0 0"/>
+                <origin xyz="0 0 0" rpy="${pi/2} 0 0"/>
                 <geometry>
-                    <mesh filename="${mesh}" scale="${mesh_scale} ${mesh_scale} ${mesh_scale}"/>
+                    <cylinder radius="0.06" length="0.04" />
                 </geometry>
             </collision>
+            <xacro:inertial_cylinder mass="0.1" radius="0.06" length="0.04">
+                <origin xyz="0 0 0" rpy="${pi/2} 0 0"/>
+            </xacro:inertial_cylinder>
             <gazebo>
                 <mu1>0.2</mu1>       <!-- lateral friction -->
@@ -41,27 +39,7 @@
     </xacro:macro>
     <!-- Four wheels -->
-    <xacro:wheel
-        name="wheel_rear_right"
-        joint_origin_xyz="0.105 -0.104 -0.0183"
-        link_xyz="-0.105 0.104 0.0183"
-        mesh="package://quac/meshes/wheel.stl"
-        />
-    <xacro:wheel
-        name="wheel_front_right"
-        joint_origin_xyz="0.105 0.104 -0.0183"
-        link_xyz="-0.105 -0.104 0.0183"
-        mesh="package://quac/meshes/wheel_2.stl"
-        />
-    <xacro:wheel
-        name="wheel_front_left"
-        joint_origin_xyz="-0.105 0.104 -0.0183"
-        link_xyz="0.105 -0.104 0.0183"
-        mesh="package://quac/meshes/wheel_3.stl"
-        />
-    <xacro:wheel
-        name="wheel_rear_left"
-        joint_origin_xyz="-0.105 -0.104 -0.0183"
-        link_xyz="0.105 0.104 0.0183"
-        mesh="package://quac/meshes/wheel_4.stl"
-        />
+    <xacro:wheel name="wheel_front_left" xyz="0.1075 0.1005 -0.03705" />
+    <xacro:wheel name="wheel_front_right" xyz="0.1075 -0.1005 -0.03705" />
+    <xacro:wheel name="wheel_rear_left" xyz="-0.1075 0.1005 -0.03705" />
+    <xacro:wheel name="wheel_rear_right" xyz="-0.1075 -0.1005 -0.03705" />
 </robot>
