Commit message: ros2 control org + launch args

File: description/gazebo.xacro (robot description, xacro)
@@ -2,7 +2,4 @@
 <robot xmlns:xacro="http://www.ros.org/wiki/xacro">
     <ros2_control name="GazeboSystemWheels" type="system">
-        <hardware>
-            <plugin>gz_ros2_control/GazeboSimSystem</plugin>
-        </hardware>
          <joint name="wheel_front_left_joint">
             <command_interface name="velocity"/>
@@ -52,40 +49,5 @@
         </joint>
     </ros2_control>
-    <gazebo>
-        <plugin name="gz_ros2_control::GazeboSimROS2ControlPlugin" filename="libgz_ros2_control-system.so">
-            <ros>
-                <namespace>quac</namespace>
-                <remapping>/robot_description:=robot_description</remapping>
-                <remapping>/tf:=tf</remapping>
-                <remapping>/clock:=clock</remapping>
-                <remapping>diff_drive_controller/cmd_vel:=cmd_vel</remapping>
-                <remapping>diff_drive_controller/odom:=odom</remapping>
-            </ros>
-            <parameters>$(find quac)/config/controllers.yaml</parameters>
-            <parameters>$(find quac)/config/gz_sim_time.yaml</parameters>
-        </plugin>
-    </gazebo>
-    <gazebo reference="lidar">
-        <material>Gazebo/Red</material>
-        <sensor name="laser" type="gpu_lidar">
-            <pose> 0 0 0 0 0 0 </pose>
-            <visualize>false</visualize>
-            <update_rate>10</update_rate>
-            <lidar>
-                <scan>
-                    <horizontal>
-                        <samples>360</samples>
-                        <min_angle>-3.14</min_angle>
-                        <max_angle>3.14</max_angle>
-                    </horizontal>
-                </scan>
-                <range>
-                    <min>0.3</min>
-                    <max>12</max>
-                </range>
-            </lidar>
-            <topic>scan</topic>
-            <gz_frame_id>lidar</gz_frame_id>
-        </sensor>
+    <gazebo reference="rear_camera">
     </gazebo>
 </robot>

File: description/robot.urdf.xacro (robot description, xacro)
@@ -7,11 +7,5 @@
     <xacro:include filename="urdf/wheels.xacro" />
     <xacro:include filename="urdf/arm.xacro" />
-    <xacro:arg name="sim_mode" default="false"/>
-    <xacro:if value="$(arg sim_mode)">
-        <xacro:include filename="gazebo.xacro" />
-    </xacro:if>
-    <xacro:unless value="$(arg sim_mode)">
-        <xacro:include filename="ros2_control.xacro" />
-    </xacro:unless>
+    <xacro:include filename="ros2_control.xacro" />
     <link name="base_link"/>
     <joint name="base_footprint_joint" type="fixed">

File: description/ros2_control.xacro (robot description, xacro)
@@ -1,110 +1,153 @@
 <?xml version="1.0"?>
 <robot xmlns:xacro="http://www.ros.org/wiki/xacro">
-    <ros2_control name="wheel_ddsm115_control" type="system">
-        <xacro:arg name="disable_wheels" default="false"/>
-        <xacro:if value="$(arg disable_wheels)">
-            <hardware>
-                <plugin>mock_components/GenericSystem</plugin>
-            </hardware>
-        </xacro:if>
-        <xacro:unless value="$(arg disable_wheels)">
-            <hardware>
-                <plugin>quac_hardware/DDSM115</plugin>
-                <param name="port">/dev/ttyUSB1</param>
-                <param name="act">1</param>
-                <param name="feedback">true</param>
-            </hardware>
-        </xacro:unless>
-        <joint name="wheel_front_left_joint">
-            <command_interface name="velocity"/>
-            <state_interface name="position"/>
-            <state_interface name="velocity"/>
-            <param name="id">4</param>
-            <param name="scalar">1</param>
-        </joint>
-        <joint name="wheel_front_right_joint">
-            <command_interface name="velocity"/>
-            <state_interface name="position"/>
-            <state_interface name="velocity"/>
-            <param name="id">1</param>
-            <param name="scalar">-1</param>
-        </joint>
-        <joint name="wheel_rear_left_joint">
-            <command_interface name="velocity"/>
-            <state_interface name="position"/>
-            <state_interface name="velocity"/>
-            <param name="id">3</param>
-            <param name="scalar">1</param>
-        </joint>
-        <joint name="wheel_rear_right_joint">
-            <command_interface name="velocity"/>
-            <state_interface name="position"/>
-            <state_interface name="velocity"/>
-            <param name="id">2</param>
-            <param name="scalar">-1</param>
-        </joint>
+    <xacro:arg name="sim_mode" default="false"/>
+    <xacro:arg name="disable_wheels" default="false"/>
+    <xacro:arg name="disable_arm" default="false"/>
+    <!-- WHEELS -->
+    <ros2_control name="wheel_control" type="system">
+        <hardware>
+            <xacro:if value="$(arg sim_mode)">
+                <plugin>gz_ros2_control/GazeboSimSystem</plugin>
+            </xacro:if>
+            <xacro:unless value="$(arg sim_mode)">
+                <xacro:unless value="$(arg disable_wheels)">
+                    <plugin>quac_hardware/DDSM115</plugin>
+                    <param name="port">/dev/ttyUSB1</param>
+                    <param name="act">1</param>
+                    <param name="feedback">true</param>
+                </xacro:unless>
+                <xacro:if value="$(arg disable_wheels)">
+                    <plugin>mock_components/GenericSystem</plugin>
+                </xacro:if>
+            </xacro:unless>
+        </hardware>
+        <xacro:macro name="wheel_joint" params="name id scalar">
+            <joint name="${name}">
+                <command_interface name="velocity"/>
+                <state_interface name="position"/>
+                <state_interface name="velocity"/>
+                <param name="id">${id}</param>
+                <param name="scalar">${scalar}</param>
+            </joint>
+        </xacro:macro>
+        <xacro:wheel_joint name="wheel_front_left_joint" id="4" scalar="1"/>
+        <xacro:wheel_joint name="wheel_front_right_joint" id="1" scalar="-1"/>
+        <xacro:wheel_joint name="wheel_rear_left_joint" id="3" scalar="1"/>
+        <xacro:wheel_joint name="wheel_rear_right_joint" id="2" scalar="-1"/>
     </ros2_control>
-    <ros2_control name="arm_waveshare_servos_control" type="system">
-        <xacro:arg name="disable_arm" default="false"/>
-        <xacro:if value="$(arg disable_arm)">
-            <hardware>
-                <plugin>mock_components/GenericSystem</plugin>
-            </hardware>
-        </xacro:if>
-        <xacro:unless value="$(arg disable_arm)">
-            <hardware>
-                <plugin>quac_hardware/WaveshareServos</plugin>
-                <param name="crawler_arm_param_hw_start_duration_sec">0</param>
-                <param name="crawler_arm_hw_stop_duration_sec">3.0</param>
-                <param name="crawler_arm_hw_slowdown">100</param>
-            </hardware>
-        </xacro:unless>
-        <joint name="arm_servo_0_joint">
-            <param name="id">5</param>
-            <param name="type">pos</param>
-            <param name="offset">1.570796</param>
-            <command_interface name="position"/>
-            <param name="pos_min">-1.570796</param>
-            <param name="pos_max">1.570796</param>
-            <command_interface name="velocity"/>
-            <param name="vel_min">-9.2</param>
-            <param name="vel_max">9.2</param>
-            <state_interface name="position"/>
-            <state_interface name="velocity"/>
-            <state_interface name="torque"/>
-            <state_interface name="temperature"/>
-        </joint>
-        <joint name="arm_servo_1_joint">
-            <param name="id">6</param>
-            <param name="type">pos</param>
-            <param name="inverted">true</param>
-            <param name="offset">1.8</param>
-            <command_interface name="position"/>
-            <param name="pos_min">-0.8</param>
-            <param name="pos_max">1.570796</param>
-            <command_interface name="velocity"/>
-            <param name="vel_min">-9.2</param>
-            <param name="vel_max">9.2</param>
-            <state_interface name="position"/>
-            <state_interface name="velocity"/>
-            <state_interface name="torque"/>
-            <state_interface name="temperature"/>
-        </joint>
-        <joint name="gripper_servo_joint">
-            <param name="id">1</param>
-            <param name="type">pos</param>
-            <param name="inverted">true</param>
-            <param name="offset">1.75</param>
-            <command_interface name="position"/>
-            <param name="pos_min">0</param>
-            <param name="pos_max">1.7</param>
-            <command_interface name="velocity"/>
-            <param name="vel_min">-9.2</param>
-            <param name="vel_max">9.2</param>
-            <state_interface name="position"/>
-            <state_interface name="velocity"/>
-            <state_interface name="torque"/>
-            <state_interface name="temperature"/>
-        </joint>
+    <!-- ARM -->
+    <ros2_control name="arm_control" type="system">
+        <hardware>
+            <xacro:if value="$(arg sim_mode)">
+                <plugin>gz_ros2_control/GazeboSimSystem</plugin>
+            </xacro:if>
+            <xacro:unless value="$(arg sim_mode)">
+                <xacro:unless value="$(arg disable_arm)">
+                    <plugin>quac_hardware/WaveshareServos</plugin>
+                    <param name="crawler_arm_param_hw_start_duration_sec">0</param>
+                    <param name="crawler_arm_hw_stop_duration_sec">3.0</param>
+                    <param name="crawler_arm_hw_slowdown">100</param>
+                </xacro:unless>
+                <xacro:if value="$(arg disable_arm)">
+                    <plugin>mock_components/GenericSystem</plugin>
+                </xacro:if>
+            </xacro:unless>
+        </hardware>
+        <xacro:macro name="arm_joint" params="name id inverted offset pos_min pos_max">
+            <joint name="${name}">
+                <param name="id">${id}</param>
+                <param name="type">pos</param>
+                <param name="inverted">${inverted}</param>
+                <param name="offset">${offset}</param>
+                <command_interface name="position"/>
+                <param name="pos_min">${pos_min}</param>
+                <param name="pos_max">${pos_max}</param>
+                <command_interface name="velocity"/>
+                <param name="vel_min">-9.2</param>
+                <param name="vel_max">9.2</param>
+                <state_interface name="position"/>
+                <state_interface name="velocity"/>
+                <state_interface name="torque"/>
+                <state_interface name="temperature"/>
+            </joint>
+        </xacro:macro>
+        <xacro:arm_joint name="arm_servo_0_joint"   id="5" inverted="false" offset="${pi/2}" pos_min="${-pi/2}" pos_max="${pi/2}"/>
+        <xacro:arm_joint name="arm_servo_1_joint"   id="6" inverted="true"  offset="1.8"     pos_min="-0.8"     pos_max="${pi/2}"/>
+        <xacro:arm_joint name="gripper_servo_joint" id="1" inverted="true"  offset="1.75"    pos_min="0"        pos_max="1.7" />
     </ros2_control>
+    <!-- EXTRA GAZEBO PLUGIN AND SENSORS -->
+    <gazebo>
+        <plugin name="gz_ros2_control::GazeboSimROS2ControlPlugin" filename="libgz_ros2_control-system.so">
+            <ros>
+                <namespace>quac</namespace>
+                <remapping>/robot_description:=robot_description</remapping>
+                <remapping>/tf:=tf</remapping>
+                <remapping>/clock:=clock</remapping>
+                <remapping>diff_drive_controller/cmd_vel:=cmd_vel</remapping>
+                <remapping>diff_drive_controller/odom:=odom</remapping>
+            </ros>
+            <parameters>$(find quac)/config/controllers.yaml</parameters>
+            <parameters>$(find quac)/config/gz_sim_time.yaml</parameters>
+        </plugin>
+    </gazebo>
+    <gazebo reference="lidar">
+        <material>Gazebo/Red</material>
+        <sensor name="lidar_sim" type="gpu_lidar">
+            <pose> 0 0 0 0 0 0 </pose>
+            <visualize>false</visualize>
+            <update_rate>10</update_rate>
+            <lidar>
+                <scan>
+                    <horizontal>
+                        <samples>360</samples>
+                        <min_angle>-3.14</min_angle>
+                        <max_angle>3.14</max_angle>
+                    </horizontal>
+                </scan>
+                <range>
+                    <min>0.3</min>
+                    <max>12</max>
+                </range>
+            </lidar>
+            <topic>scan</topic>
+            <gz_frame_id>lidar</gz_frame_id>
+        </sensor>
+    </gazebo>
+    <xacro:macro name="cam_sim" params="frame">
+        <gazebo reference="${frame}">
+            <sensor name="${frame}_sim" type="rgbd_camera">
+                <always_on>true</always_on>
+                <visualize>true</visualize>
+                <update_rate>10</update_rate>
+                <topic>${frame}</topic>
+                <gz_frame_id>${frame}</gz_frame_id>
+                <camera>
+                <horizontal_fov>1.48702</horizontal_fov>
+                <image>
+                    <width>640</width>
+                    <height>480</height>
+                </image>
+                <clip>
+                    <near>0.05</near>
+                    <far>3</far>
+                </clip>
+                </camera>
+                <baseline>0.2</baseline>
+                <pointCloudCutoff>0.5</pointCloudCutoff>
+                <pointCloudCutoffMax>3.0</pointCloudCutoffMax>
+                <distortionK1>0</distortionK1>
+                <distortionK2>0</distortionK2>
+                <distortionK3>0</distortionK3>
+                <distortionT1>0</distortionT1>
+                <distortionT2>0</distortionT2>
+                <CxPrime>0</CxPrime>
+                <Cx>0</Cx>
+                <Cy>0</Cy>
+                <focalLength>0</focalLength>
+                <hackBaseline>0</hackBaseline>
+            </sensor>
+        </gazebo>
+    </xacro:macro>
+    <xacro:cam_sim frame="front_camera"/>
+    <xacro:cam_sim frame="rear_camera"/>
 </robot>

File: description/urdf/arm.xacro (robot description, xacro)
@@ -91,3 +91,9 @@
         </xacro:inertial_cylinder>
     </link>
+    <joint name="front_camera_joint" type="fixed">
+        <parent link="gripper_gear"/>
+        <child link="front_camera"/>
+        <origin xyz="0.0 0.0 0.0" rpy="0 0 0"/>
+    </joint>
+    <link name="front_camera"/>
 </robot>

File: description/urdf/chassis.xacro (robot description, xacro)
@@ -47,3 +47,9 @@
     </joint>
     <link name="lidar"/>
+    <joint name="rear_camera_joint" type="fixed">
+        <parent link="chassis"/>
+        <child link="rear_camera"/>
+        <origin xyz="-0.09 0.0 0.1" rpy="0 0 ${pi}"/>
+    </joint>
+    <link name="rear_camera"/>
 </robot>
