Commit message: stuff

File: quac/description/ros2_control.xacro (robot description, xacro)
@@ -92,5 +92,5 @@
         </plugin>
     </gazebo>
-    <gazebo reference="lidar">
+    <gazebo reference="laser">
         <material>Gazebo/Red</material>
         <sensor name="lidar_sim" type="gpu_lidar">
@@ -112,5 +112,5 @@
             </lidar>
             <topic>scan</topic>
-            <gz_frame_id>lidar</gz_frame_id>
+            <gz_frame_id>laser</gz_frame_id>
         </sensor>
     </gazebo>

File: quac/description/urdf/chassis.xacro (robot description, xacro)
@@ -38,13 +38,10 @@
         <gravity>true</gravity>
     </gazebo>
-    <material name="lidar_material">
-        <color rgba="0.8 0.2 0.2 1.0" />
-    </material>
-    <joint name="lidar_joint" type="fixed">
+    <joint name="laser_joint" type="fixed">
         <parent link="chassis"/>
-        <child link="lidar"/>
+        <child link="laser"/>
         <origin xyz="-0.02 0.0 0.15" rpy="0 0 0"/>
     </joint>
-    <link name="lidar"/>
+    <link name="laser"/>
     <joint name="rear_camera_joint" type="fixed">
         <parent link="chassis"/>

Commit message: not working but almost

File: quac/description/ros2_control.xacro (robot description, xacro)
@@ -73,7 +73,7 @@
             </joint>
         </xacro:macro>
-        <xacro:arm_joint name="arm_servo_0_joint"   id="5" inverted="false" offset="${pi/2}" pos_min="${-pi/2}" pos_max="${pi/2}"/>
-        <xacro:arm_joint name="arm_servo_1_joint"   id="6" inverted="true"  offset="1.8"     pos_min="-0.8"     pos_max="${pi/2}"/>
-        <xacro:arm_joint name="gripper_servo_joint" id="1" inverted="true"  offset="1.75"    pos_min="0"        pos_max="1.7" />
+        <xacro:arm_joint name="arm_servo_0_joint"   id="5" inverted="false" offset="${pi}" pos_min="${-pi/2}" pos_max="${pi/2}"/>
+        <xacro:arm_joint name="arm_servo_1_joint"   id="6" inverted="true"  offset="1.8"   pos_min="-0.8"     pos_max="${pi/2}"/>
+        <xacro:arm_joint name="gripper_servo_joint" id="1" inverted="true"  offset="1.75"  pos_min="0"        pos_max="1.7" />
     </ros2_control>
     <!-- EXTRA GAZEBO PLUGIN AND SENSORS -->

File: quac/description/urdf/chassis.xacro (robot description, xacro)
@@ -41,5 +41,5 @@
         <parent link="chassis"/>
         <child link="laser"/>
-        <origin xyz="-0.02 0.0 0.15" rpy="0 0 0"/>
+        <origin xyz="-0.02 0.0 0.15" rpy="0 0 ${pi}"/>
     </joint>
     <link name="laser"/>
