Commit message: frames + realsense model

File: src/quac/description/urdf/arm.xacro (robot description, xacro)
@@ -94,9 +94,6 @@
         </xacro:inertial_cylinder>
     </link>
-    <joint name="camera_front_joint" type="fixed">
-        <parent link="gripper_gear"/>
-        <child link="camera_front"/>
-        <origin xyz="0.0 0.0 0.0" rpy="0 0 0"/>
-    </joint>
-    <link name="camera_front"/>
+    <xacro:sensor_d435 parent="gripper_servo" name="camera_front" use_nominal_extrinsics="true" add_plug="false" use_mesh="true">
+        <origin xyz="0 0 0" rpy="0 0 0"/>
+    </xacro:sensor_d435>
 </robot>

File: src/quac/description/urdf/chassis.xacro (robot description, xacro)
@@ -44,14 +44,5 @@
     </joint>
     <link name="imu"/>
-    <!-- <joint name="camera_back_joint" type="fixed">
-        <parent link="chassis"/>
-        <child link="camera_back"/>
-        <origin xyz="-0.09 0.0 0.1" rpy="0 0 ${pi}"/>
-    </joint>
-    <link name="camera_back"/> -->
-    <xacro:arg name="use_nominal_extrinsics" default="false"/>
-    <xacro:arg name="add_plug" default="true" />
-    <xacro:arg name="use_mesh" default="true" />
-    <xacro:sensor_d435 parent="chassis" name="camera_back" use_nominal_extrinsics="$(arg use_nominal_extrinsics)" add_plug="$(arg add_plug)" use_mesh="$(arg use_mesh)">
+    <xacro:sensor_d435 parent="chassis" name="camera_back" use_nominal_extrinsics="true" add_plug="false" use_mesh="true">
         <origin xyz="-0.09 0.0 0.1" rpy="0 0 ${pi}"/>
     </xacro:sensor_d435>
