Commit message: new model

File: src/quac/description/robot.urdf.xacro (robot description, xacro)
@@ -1,8 +1,9 @@
 <?xml version="1.0"?>
 <robot xmlns:xacro="http://www.ros.org/wiki/xacro"  name="quac_robot">
-    <xacro:property name="mesh_scale" value="0.001"/>
+    <xacro:property name="mesh_scale" value="1"/>
     <xacro:include filename="urdf/inertial_macros.xacro" />
     <xacro:include filename="urdf/servo.xacro" />
     <xacro:include filename="urdf/d435.xacro" />
+    <xacro:include filename="urdf/oak_d_lite.xacro" />
     <xacro:include filename="urdf/version_6/chassis.xacro" />
     <xacro:unless value="$(arg sim_mode)">

File: src/quac/description/urdf/version_6/arm.xacro (robot description, xacro)
@@ -1,4 +1,10 @@
 <?xml version="1.0"?>
 <robot xmlns:xacro="http://www.ros.org/wiki/xacro">
+<material name="gripper_material">
+    <color rgba="0.7 0.2 0.2 1.0" />
+</material>
+<material name="arm_material">
+    <color rgba="0.7 0.7 0.7 1.0" />
+</material>
     <joint name="arm_servo_0_joint" type="continuous">
         <parent link="chassis"/>
@@ -8,13 +14,10 @@
     </joint>
     <link name="arm_segment_1">
-        <xacro:inertial_box mass="0.1" x="0.10" y="0.04" z="0.04">
-            <origin xyz="0 0 0" rpy="0 0 0"/>
-        </xacro:inertial_box>
         <visual>
-            <origin xyz="0 0 0" rpy="0 0 0"/>
+            <origin xyz="0 0 0" rpy="${-pi/2} 0 0"/>
             <geometry>
-                <mesh filename="package://quac/meshes/version_6/arm_segment_1.glb" scale="${mesh_scale} ${mesh_scale} ${mesh_scale}"/>
+                <mesh filename="package://quac/meshes/version_6/arm_segment_1_reduced.stl" scale="${mesh_scale} ${mesh_scale} ${mesh_scale}"/>
             </geometry>
-            <material name="chassis_material"/>
+            <material name="arm_material"/>
         </visual>
     </link>
@@ -26,39 +29,73 @@
     </joint>
     <link name="arm_segment_2">
-        <xacro:inertial_box mass="0.1" x="0.10" y="0.04" z="0.04">
-            <origin xyz="0 0 0" rpy="0 0 0"/>
-        </xacro:inertial_box>
         <visual>
-            <origin xyz="0 0 0" rpy="0 0 0"/>
+            <origin xyz="0 0 0" rpy="${-pi/2} 0 0"/>
             <geometry>
-                <mesh filename="package://quac/meshes/version_6/arm_segment_2.glb" scale="${mesh_scale} ${mesh_scale} ${mesh_scale}"/>
+                <mesh filename="package://quac/meshes/version_6/arm_segment_2_reduced.stl" scale="${mesh_scale} ${mesh_scale} ${mesh_scale}"/>
             </geometry>
-            <material name="chassis_material"/>
+            <material name="arm_material"/>
         </visual>
     </link>
+    <xacro:sensor_d435 parent="arm_segment_2" name="camera_gripper" use_nominal_extrinsics="true">
+        <origin xyz="0.09 0.025 0.025" rpy="${-pi/2} 0 0"/>
+    </xacro:sensor_d435>
     <joint name="gripper_servo_joint" type="continuous">
         <parent link="arm_segment_2" />
         <child link="gripper_gear" />
-        <origin xyz="0.05 0.04 0" rpy="${-pi/2} 0 0"/>
+        <origin xyz="0.0483 0.04 -0.0125" rpy="${-pi/2} 0 0"/>
         <axis xyz="0 0 1" />
     </joint>
-    <link name="gripper_gear">
-        <visual>
-            <geometry>
-                <cylinder radius="0.02" length="0.02" />
-            </geometry>
-            <material name="gripper_material" />
-        </visual>
-        <collision>
-            <geometry>
-                <cylinder radius="0.02" length="0.02" />
-            </geometry>
-        </collision>
-        <xacro:inertial_cylinder mass="0.1" length="0.02" radius="0.02">
-            <origin xyz="0 0 0" rpy="0 0 0"/>
-        </xacro:inertial_cylinder>
-    </link>
-    <xacro:sensor_d435 parent="arm_segment_2" name="camera_front" use_nominal_extrinsics="true">
-        <origin xyz="0.095 0.016 0" rpy="${-pi/2} 0 0"/>
-    </xacro:sensor_d435>
+    <link name="gripper_gear"></link>
+    <xacro:macro name="gripper_side" params="side multiplier">
+        <joint name="gripper_${side}_back_piece_joint" type="continuous">
+            <parent link="arm_segment_2" />
+            <child link="gripper_${side}_back_piece" />
+            <origin xyz="0.048 0.015 ${multiplier * 0.0315}" rpy="${-pi/2} 0 0"/>
+            <mimic joint="gripper_servo_joint" multiplier="${-multiplier}" offset="${multiplier * pi/2}"/>
+            <axis xyz="0 0 1" />
+        </joint>
+        <link name="gripper_${side}_back_piece">
+            <visual>
+                <origin xyz="0 0 0" rpy="0 0 ${pi/2+multiplier*pi/2}"/>
+                <geometry>
+                    <mesh filename="package://quac/meshes/version_6/gripper_back_piece.stl" scale="${mesh_scale} ${mesh_scale} ${mesh_scale}"/>
+                </geometry>
+                <material name="gripper_material"/>
+            </visual>
+        </link>
+        <joint name="gripper_${side}_front_piece_joint" type="continuous">
+            <parent link="arm_segment_2" />
+            <child link="gripper_${side}_front_piece" />
+            <origin xyz="0.069 0.0045 ${multiplier * 0.0105}" rpy="${-pi/2} 0 0"/>
+            <mimic joint="gripper_servo_joint" multiplier="${-multiplier}" offset="${multiplier * pi/2}"/>
+            <axis xyz="0 0 1" />
+        </joint>
+        <link name="gripper_${side}_front_piece">
+            <visual>
+                <origin xyz="0 0 0" rpy="0 0 ${pi/2+multiplier*pi/2}"/>
+                <geometry>
+                    <mesh filename="package://quac/meshes/version_6/gripper_front_piece.stl" scale="${mesh_scale} ${mesh_scale} ${mesh_scale}"/>
+                </geometry>
+                <material name="gripper_material"/>
+            </visual>
+        </link>
+        <joint name="gripper_${side}_joint" type="continuous">
+            <parent link="gripper_${side}_back_piece" />
+            <child link="gripper_${side}" />
+            <origin xyz="0.0 ${-multiplier * 0.043} 0.006" rpy="0 0 0"/>
+            <mimic joint="gripper_servo_joint" multiplier="${multiplier}" offset="${-multiplier * pi/2}"/>
+            <axis xyz="0 0 1" />
+        </joint>
+        <link name="gripper_${side}">
+            <visual>
+                <origin xyz="0 0 0" rpy="0 0 0"/>
+                <geometry>
+                    <mesh filename="package://quac/meshes/version_6/gripper_${side}.stl" scale="${mesh_scale} ${mesh_scale} ${mesh_scale}"/>
+                </geometry>
+                <material name="gripper_material"/>
+            </visual>
+        </link>
+    </xacro:macro>
+    <xacro:gripper_side side="left" multiplier="-1.0" />
+    <xacro:gripper_side side="right" multiplier="1.0" />
 </robot>

File: src/quac/description/urdf/version_6/chassis.xacro (robot description, xacro)
@@ -5,10 +5,4 @@
     <material name="chassis_material">
         <color rgba="1.0 1.0 1.0 1.0" />
-    </material>
-    <material name="wheel_material">
-        <color rgba="0.6 0.6 0.6 1.0" />
-    </material>
-    <material name="gripper_material">
-        <color rgba="0.8 0.0 0.0 1.0" />
     </material>
     <joint name="chassis_joint" type="fixed">
@@ -24,7 +18,7 @@
         </inertial>
         <visual>
-            <origin xyz="0 0 0" rpy="${pi/2} 0 0"/>
+            <origin xyz="0 0 0" rpy="0 0 0"/>
             <geometry>
-                <mesh filename="package://quac/meshes/version_6/chassis.glb" scale="${mesh_scale} ${mesh_scale} ${mesh_scale}"/>
+                <mesh filename="package://quac/meshes/version_6/chassis_reduced.stl" scale="${mesh_scale} ${mesh_scale} ${mesh_scale}"/>
             </geometry>
             <material name="chassis_material"/>
@@ -34,5 +28,5 @@
         <parent link="chassis"/>
         <child link="laser"/>
-        <origin xyz="-0.035 0.0 0.122" rpy="0 0 ${pi/2}"/>
+        <origin xyz="-0.035 0.0 0.127" rpy="0 0 ${pi/2}"/>
     </joint>
     <link name="laser"/>
@@ -46,3 +40,4 @@
         <origin xyz="-0.09 0.0 0.09" rpy="0 0 ${pi}"/>
     </xacro:sensor_d435>
+	<xacro:oak_d_lite camera_name="camera_front" parent="chassis" cam_pos_x="0.16" cam_pos_y="0" cam_pos_z="-0.015" cam_roll="0" cam_pitch="0" cam_yaw="0"/>
 </robot>

File: src/quac/description/urdf/version_6/wheels.xacro (robot description, xacro)
@@ -1,4 +1,7 @@
 <?xml version="1.0"?>
 <robot xmlns:xacro="http://www.ros.org/wiki/xacro">
+    <material name="wheel_material">
+        <color rgba="0.6 0.6 0.6 1.0" />
+    </material>
     <xacro:macro name="wheel" params="name xyz visual_rpy collision_xyz">
         <joint name="${name}_joint" type="continuous">
@@ -12,5 +15,5 @@
                 <origin xyz="0 0 0" rpy="${visual_rpy}"/>
                 <geometry>
-                    <mesh filename="package://quac/meshes/version_6/wheel.glb" scale="${mesh_scale} ${mesh_scale} ${mesh_scale}"/>
+                    <mesh filename="package://quac/meshes/version_6/wheel_reduced.stl" scale="${mesh_scale} ${mesh_scale} ${mesh_scale}"/>
                 </geometry>
                 <material name="wheel_material"/>
@@ -36,7 +39,7 @@
     </xacro:macro>
     <!-- Four wheels -->
-    <xacro:wheel name="wheel_front_left" xyz="0.114 0.0615 -0.074" visual_rpy="0 ${pi/2} 0" collision_xyz="0 0.03 0" />
-    <xacro:wheel name="wheel_front_right" xyz="0.114 -0.0615 -0.074" visual_rpy="0 ${pi/2} ${pi}" collision_xyz="0 -0.03 0" />
-    <xacro:wheel name="wheel_rear_left" xyz="-0.114 0.0615 -0.074" visual_rpy="0 ${pi/2} 0" collision_xyz="0 0.03 0" />
-    <xacro:wheel name="wheel_rear_right" xyz="-0.114 -0.0615 -0.074" visual_rpy="0 ${pi/2} ${pi}" collision_xyz="0 -0.03 0" />
+    <xacro:wheel name="wheel_front_left" xyz="0.109 0.063 -0.079" visual_rpy="0 0 ${pi}" collision_xyz="0 0.03 0" />
+    <xacro:wheel name="wheel_front_right" xyz="0.109 -0.063 -0.079" visual_rpy="0 0 0" collision_xyz="0 -0.03 0" />
+    <xacro:wheel name="wheel_rear_left" xyz="-0.109 0.063 -0.079" visual_rpy="0 0 ${pi}" collision_xyz="0 0.03 0" />
+    <xacro:wheel name="wheel_rear_right" xyz="-0.109 -0.063 -0.079" visual_rpy="0 0 0" collision_xyz="0 -0.03 0" />
 </robot>
