Commit message: new launch + work on camera app

File: src/quac/description/gazebo.xacro (robot description, xacro)
@@ -49,5 +49,5 @@
         </joint>
     </ros2_control>
-    <gazebo reference="rear_camera">
+    <gazebo reference="camera_back">
     </gazebo>
 </robot>

File: src/quac/description/ros2_control.xacro (robot description, xacro)
@@ -89,5 +89,5 @@
                 <remapping>arm_position_controller/joint_trajectory:=arm_joint_trajectory</remapping>
             </ros>
-            <parameters>$(find quac)/config/control.yaml</parameters>
+            <parameters>$(find quac)/config/controllers.yaml</parameters>
             <parameters>$(find quac)/config/gz_sim_time.yaml</parameters>
         </plugin>
@@ -151,5 +151,5 @@
         </gazebo>
     </xacro:macro>
-    <xacro:cam_sim frame="front_camera"/>
-    <xacro:cam_sim frame="rear_camera"/>
+    <xacro:cam_sim frame="camera_font"/>
+    <xacro:cam_sim frame="camera_back"/>
 </robot>

File: src/quac/description/urdf/arm.xacro (robot description, xacro)
@@ -91,9 +91,9 @@
         </xacro:inertial_cylinder>
     </link>
-    <joint name="front_camera_joint" type="fixed">
+    <joint name="camera_font_joint" type="fixed">
         <parent link="gripper_gear"/>
-        <child link="front_camera"/>
+        <child link="camera_font"/>
         <origin xyz="0.0 0.0 0.0" rpy="0 0 0"/>
     </joint>
-    <link name="front_camera"/>
+    <link name="camera_font"/>
 </robot>

File: src/quac/description/urdf/chassis.xacro (robot description, xacro)
@@ -38,9 +38,9 @@
     </joint>
     <link name="laser"/>
-    <joint name="rear_camera_joint" type="fixed">
+    <joint name="camera_back_joint" type="fixed">
         <parent link="chassis"/>
-        <child link="rear_camera"/>
+        <child link="camera_back"/>
         <origin xyz="-0.09 0.0 0.1" rpy="0 0 ${pi}"/>
     </joint>
-    <link name="rear_camera"/>
+    <link name="camera_back"/>
 </robot>

Commit message: fixes + gazebo lidar

File: src/quac/description/gazebo.xacro (robot description, xacro)
@@ -2,24 +2,24 @@
 <robot xmlns:xacro="http://www.ros.org/wiki/xacro">
     <ros2_control name="GazeboSystemWheels" type="system">
-         <joint name="wheel_front_left_joint">
-            <command_interface name="velocity"/>
-            <state_interface name="position"/>
-            <state_interface name="velocity"/>
-        </joint>
-        <joint name="wheel_front_right_joint">
-            <command_interface name="velocity"/>
-            <state_interface name="position"/>
-            <state_interface name="velocity"/>
-        </joint>
-        <joint name="wheel_rear_left_joint">
-            <command_interface name="velocity"/>
-            <state_interface name="position"/>
-            <state_interface name="velocity"/>
-        </joint>
-        <joint name="wheel_rear_right_joint">
-            <command_interface name="velocity"/>
-            <state_interface name="position"/>
-            <state_interface name="velocity"/>
-        </joint>
+    <joint name="wheel_front_left_joint">
+        <command_interface name="velocity"/>
+        <state_interface name="position"/>
+        <state_interface name="velocity"/>
+    </joint>
+    <joint name="wheel_front_right_joint">
+        <command_interface name="velocity"/>
+        <state_interface name="position"/>
+        <state_interface name="velocity"/>
+    </joint>
+    <joint name="wheel_rear_left_joint">
+        <command_interface name="velocity"/>
+        <state_interface name="position"/>
+        <state_interface name="velocity"/>
+    </joint>
+    <joint name="wheel_rear_right_joint">
+        <command_interface name="velocity"/>
+        <state_interface name="position"/>
+        <state_interface name="velocity"/>
+    </joint>
     </ros2_control>
     <ros2_control name="GazeboSystemServos" type="system">
@@ -49,5 +49,86 @@
         </joint>
     </ros2_control>
-    <gazebo reference="camera_back">
+    <gazebo>
+        <plugin name="gz_ros2_control::GazeboSimROS2ControlPlugin" filename="libgz_ros2_control-system.so">
+            <ros>
+                <namespace>quac</namespace>
+                <remapping>/robot_description:=robot_description</remapping>
+                <remapping>/tf:=tf</remapping>
+                <remapping>/clock:=clock</remapping>
+                <remapping>diff_drive_controller/cmd_vel_unstamped:=cmd_vel</remapping>
+                <remapping>diff_drive_controller/odom:=odom</remapping>
+                <remapping>arm_position_controller/joint_trajectory:=arm_joint_trajectory</remapping>
+            </ros>
+            <parameters>$(find quac)/config/controllers.yaml</parameters>
+            <parameters>$(find quac)/config/gz_sim_time.yaml</parameters>
+        </plugin>
+    </gazebo>
+    <gazebo reference="laser">
+        <material>Gazebo/Red</material>
+        <sensor name="lidar_sim" type="gpu_lidar">
+            <pose> 0 0 0 0 0 0 </pose>
+            <visualize>false</visualize>
+            <update_rate>10</update_rate>
+            <lidar>
+                <scan>
+                    <horizontal>
+                        <samples>360</samples>
+                        <min_angle>-3.14</min_angle>
+                        <max_angle>3.14</max_angle>
+                    </horizontal>
+                </scan>
+                <range>
+                    <min>0.3</min>
+                    <max>12</max>
+                </range>
+            </lidar>
+            <topic>scan</topic>
+            <gz_frame_id>laser</gz_frame_id>
+        </sensor>
+    </gazebo>
+    <xacro:macro name="cam_sim" params="frame">
+        <gazebo reference="${frame}">
+            <sensor name="${frame}_sim" type="rgbd_camera">
+                <always_on>true</always_on>
+                <visualize>true</visualize>
+                <update_rate>10</update_rate>
+                <topic>${frame}</topic>
+                <gz_frame_id>${frame}</gz_frame_id>
+                <camera>
+                <horizontal_fov>1.48702</horizontal_fov>
+                <image>
+                    <width>640</width>
+                    <height>480</height>
+                </image>
+                <clip>
+                    <near>0.05</near>
+                    <far>3</far>
+                </clip>
+                </camera>
+                <baseline>0.2</baseline>
+                <pointCloudCutoff>0.5</pointCloudCutoff>
+                <pointCloudCutoffMax>3.0</pointCloudCutoffMax>
+                <distortionK1>0</distortionK1>
+                <distortionK2>0</distortionK2>
+                <distortionK3>0</distortionK3>
+                <distortionT1>0</distortionT1>
+                <distortionT2>0</distortionT2>
+                <CxPrime>0</CxPrime>
+                <Cx>0</Cx>
+                <Cy>0</Cy>
+                <focalLength>0</focalLength>
+                <hackBaseline>0</hackBaseline>
+            </sensor>
+        </gazebo>
+    </xacro:macro>
+    <xacro:cam_sim frame="camera_front"/>
+    <xacro:cam_sim frame="camera_back"/>
+    <gazebo reference="imu">
+        <sensor name="imu_sim" type="imu">
+            <always_on>1</always_on>
+            <update_rate>10</update_rate>
+            <visualize>true</visualize>
+            <topic>imu</topic>
+        </sensor>
     </gazebo>
 </robot>

File: src/quac/description/robot.urdf.xacro (robot description, xacro)
@@ -7,5 +7,10 @@
     <xacro:include filename="urdf/wheels.xacro" />
     <xacro:include filename="urdf/arm.xacro" />
-    <xacro:include filename="ros2_control.xacro" />
+    <xacro:unless value="$(arg sim_mode)">
+        <xacro:include filename="ros2_control.xacro" />
+    </xacro:unless>
+    <xacro:if value="$(arg sim_mode)">
+        <xacro:include filename="gazebo.xacro" />
+    </xacro:if>
     <link name="base_link"/>
     <joint name="base_footprint_joint" type="fixed">

File: src/quac/description/ros2_control.xacro (robot description, xacro)
@@ -7,17 +7,12 @@
     <ros2_control name="wheel_hardware" type="system">
         <hardware>
-            <xacro:if value="$(arg sim_mode)">
-                <plugin>gz_ros2_control/GazeboSimSystem</plugin>
+            <xacro:unless value="$(arg disable_wheels)">
+                <plugin>quac_hardware/DDSM115</plugin>
+                <param name="port">/dev/quac/wheels_rs485</param>
+                <param name="act">3</param>
+            </xacro:unless>
+            <xacro:if value="$(arg disable_wheels)">
+                <plugin>mock_components/GenericSystem</plugin>
             </xacro:if>
-            <xacro:unless value="$(arg sim_mode)">
-                <xacro:unless value="$(arg disable_wheels)">
-                    <plugin>quac_hardware/DDSM115</plugin>
-                    <param name="port">/dev/quac/wheels_rs485</param>
-                    <param name="act">1</param>
-                </xacro:unless>
-                <xacro:if value="$(arg disable_wheels)">
-                    <plugin>mock_components/GenericSystem</plugin>
-                </xacro:if>
-            </xacro:unless>
         </hardware>
         <xacro:macro name="wheel_joint" params="name id scalar">
@@ -39,19 +34,14 @@
     <ros2_control name="arm_hardware" type="system">
         <hardware>
-            <xacro:if value="$(arg sim_mode)">
-                <plugin>gz_ros2_control/GazeboSimSystem</plugin>
+            <xacro:unless value="$(arg disable_arm)">
+                <plugin>quac_hardware/WaveshareServos</plugin>
+                <param name="port">/dev/quac/arm_servos</param>
+                <param name="crawler_arm_param_hw_start_duration_sec">0</param>
+                <param name="crawler_arm_hw_stop_duration_sec">3.0</param>
+                <param name="crawler_arm_hw_slowdown">100</param>
+            </xacro:unless>
+            <xacro:if value="$(arg disable_arm)">
+                <plugin>mock_components/GenericSystem</plugin>
             </xacro:if>
-            <xacro:unless value="$(arg sim_mode)">
-                <xacro:unless value="$(arg disable_arm)">
-                    <plugin>quac_hardware/WaveshareServos</plugin>
-                    <param name="port">/dev/quac/arm_servos</param>
-                    <param name="crawler_arm_param_hw_start_duration_sec">0</param>
-                    <param name="crawler_arm_hw_stop_duration_sec">3.0</param>
-                    <param name="crawler_arm_hw_slowdown">100</param>
-                </xacro:unless>
-                <xacro:if value="$(arg disable_arm)">
-                    <plugin>mock_components/GenericSystem</plugin>
-                </xacro:if>
-            </xacro:unless>
         </hardware>
         <xacro:macro name="arm_joint" params="name id inverted offset pos_min pos_max">
@@ -77,79 +67,2 @@
         <xacro:arm_joint name="gripper_servo_joint" id="1" inverted="true"  offset="1.75"  pos_min="0"        pos_max="1.7" />
     </ros2_control>
-    <!-- EXTRA GAZEBO PLUGIN AND SENSORS -->
-    <gazebo>
-        <plugin name="gz_ros2_control::GazeboSimROS2ControlPlugin" filename="libgz_ros2_control-system.so">
-            <ros>
-                <namespace>quac</namespace>
-                <remapping>/robot_description:=robot_description</remapping>
-                <remapping>/tf:=tf</remapping>
-                <remapping>/clock:=clock</remapping>
-                <remapping>diff_drive_controller/cmd_vel_unstamped:=cmd_vel</remapping>
-                <remapping>diff_drive_controller/odom:=odom</remapping>
-                <remapping>arm_position_controller/joint_trajectory:=arm_joint_trajectory</remapping>
-            </ros>
-            <parameters>$(find quac)/config/controllers.yaml</parameters>
-            <parameters>$(find quac)/config/gz_sim_time.yaml</parameters>
-        </plugin>
-    </gazebo>
-    <gazebo reference="laser">
-        <material>Gazebo/Red</material>
-        <sensor name="lidar_sim" type="gpu_lidar">
-            <pose> 0 0 0 0 0 0 </pose>
-            <visualize>false</visualize>
-            <update_rate>10</update_rate>
-            <lidar>
-                <scan>
-                    <horizontal>
-                        <samples>360</samples>
-                        <min_angle>-3.14</min_angle>
-                        <max_angle>3.14</max_angle>
-                    </horizontal>
-                </scan>
-                <range>
-                    <min>0.3</min>
-                    <max>12</max>
-                </range>
-            </lidar>
-            <topic>scan</topic>
-            <gz_frame_id>laser</gz_frame_id>
-        </sensor>
-    </gazebo>
-    <xacro:macro name="cam_sim" params="frame">
-        <gazebo reference="${frame}">
-            <sensor name="${frame}_sim" type="rgbd_camera">
-                <always_on>true</always_on>
-                <visualize>true</visualize>
-                <update_rate>10</update_rate>
-                <topic>${frame}</topic>
-                <gz_frame_id>${frame}</gz_frame_id>
-                <camera>
-                <horizontal_fov>1.48702</horizontal_fov>
-                <image>
-                    <width>640</width>
-                    <height>480</height>
-                </image>
-                <clip>
-                    <near>0.05</near>
-                    <far>3</far>
-                </clip>
-                </camera>
-                <baseline>0.2</baseline>
-                <pointCloudCutoff>0.5</pointCloudCutoff>
-                <pointCloudCutoffMax>3.0</pointCloudCutoffMax>
-                <distortionK1>0</distortionK1>
-                <distortionK2>0</distortionK2>
-                <distortionK3>0</distortionK3>
-                <distortionT1>0</distortionT1>
-                <distortionT2>0</distortionT2>
-                <CxPrime>0</CxPrime>
-                <Cx>0</Cx>
-                <Cy>0</Cy>
-                <focalLength>0</focalLength>
-                <hackBaseline>0</hackBaseline>
-            </sensor>
-        </gazebo>
-    </xacro:macro>
-    <xacro:cam_sim frame="camera_font"/>
-    <xacro:cam_sim frame="camera_back"/>
-</robot>

File: src/quac/description/urdf/arm.xacro (robot description, xacro)
@@ -91,9 +91,9 @@
         </xacro:inertial_cylinder>
     </link>
-    <joint name="camera_font_joint" type="fixed">
+    <joint name="camera_front_joint" type="fixed">
         <parent link="gripper_gear"/>
-        <child link="camera_font"/>
+        <child link="camera_front"/>
         <origin xyz="0.0 0.0 0.0" rpy="0 0 0"/>
     </joint>
-    <link name="camera_font"/>
+    <link name="camera_front"/>
 </robot>

File: src/quac/description/urdf/chassis.xacro (robot description, xacro)
@@ -38,4 +38,10 @@
     </joint>
     <link name="laser"/>
+    <joint name="imu_joint" type="fixed">
+        <parent link="chassis"/>
+        <child link="imu"/>
+        <origin xyz="-0.02 0.04 0.145" rpy="0 0 0"/>
+    </joint>
+    <link name="imu"/>
     <joint name="camera_back_joint" type="fixed">
         <parent link="chassis"/>

Commit message: fixes

File: src/quac/description/gazebo.xacro (robot description, xacro)
@@ -2,24 +2,27 @@
 <robot xmlns:xacro="http://www.ros.org/wiki/xacro">
     <ros2_control name="GazeboSystemWheels" type="system">
-    <joint name="wheel_front_left_joint">
-        <command_interface name="velocity"/>
-        <state_interface name="position"/>
-        <state_interface name="velocity"/>
-    </joint>
-    <joint name="wheel_front_right_joint">
-        <command_interface name="velocity"/>
-        <state_interface name="position"/>
-        <state_interface name="velocity"/>
-    </joint>
-    <joint name="wheel_rear_left_joint">
-        <command_interface name="velocity"/>
-        <state_interface name="position"/>
-        <state_interface name="velocity"/>
-    </joint>
-    <joint name="wheel_rear_right_joint">
-        <command_interface name="velocity"/>
-        <state_interface name="position"/>
-        <state_interface name="velocity"/>
-    </joint>
+        <hardware>
+            <plugin>gz_ros2_control/GazeboSimSystem</plugin>
+        </hardware>
+        <joint name="wheel_front_left_joint">
+            <command_interface name="velocity"/>
+            <state_interface name="position"/>
+            <state_interface name="velocity"/>
+        </joint>
+        <joint name="wheel_front_right_joint">
+            <command_interface name="velocity"/>
+            <state_interface name="position"/>
+            <state_interface name="velocity"/>
+        </joint>
+        <joint name="wheel_rear_left_joint">
+            <command_interface name="velocity"/>
+            <state_interface name="position"/>
+            <state_interface name="velocity"/>
+        </joint>
+        <joint name="wheel_rear_right_joint">
+            <command_interface name="velocity"/>
+            <state_interface name="position"/>
+            <state_interface name="velocity"/>
+        </joint>
     </ros2_control>
     <ros2_control name="GazeboSystemServos" type="system">
@@ -130,4 +133,6 @@
             <visualize>true</visualize>
             <topic>imu</topic>
+            <enable_metrics>true</enable_metrics>
+            <gz_frame_id>imu</gz_frame_id>
         </sensor>
     </gazebo>

File: src/quac/description/ros2_control.xacro (robot description, xacro)
@@ -67,2 +67,3 @@
         <xacro:arm_joint name="gripper_servo_joint" id="1" inverted="true"  offset="1.75"  pos_min="0"        pos_max="1.7" />
     </ros2_control>
+</robot>

File: src/quac/description/urdf/arm.xacro (robot description, xacro)
@@ -27,20 +27,23 @@
         <color rgba="0.5 0.00 0.00 1.0" />
     </material>
+    <material name="yellow">
+        <color rgba="0.8 0.8 0.00 1.0" />
+    </material>
     <!-- Model -->
     <joint name="arm_base_joint" type="fixed">
         <parent link="chassis" />
         <child link="arm_servo_0_axis" />
-        <origin xyz="0.135 0.0 0.064" rpy="${pi/2} ${pi/2} 0" />
+        <origin xyz="0.135 0.0 0.064" rpy="${pi/2} 0 0" />
     </joint>
-    <xacro:servo_flipped name="arm_servo_0"/>
+    <xacro:servo name="arm_servo_0" flipped="true"/>
     <joint name="plate_0_joint" type="fixed">
         <parent link="arm_servo_0" />
         <child link="plate_0" />
-        <origin xyz="-0.058875 0.0 0.0185" rpy="0 0 0" />
+        <origin xyz="-0.0625 0.0 0.0185" rpy="0 0 0" />
     </joint>
     <joint name="plate_1_joint" type="fixed">
         <parent link="arm_servo_0" />
         <child link="plate_1" />
-        <origin xyz="-0.058875 0.0 -0.0185" rpy="0 0 0" />
+        <origin xyz="-0.0625 0.0 -0.0185" rpy="0 0 0" />
     </joint>
     <xacro:plate plate_name="plate_0"/>
@@ -49,16 +52,16 @@
         <parent link="arm_servo_0" />
         <child link="arm_servo_1" />
-        <origin xyz="-0.101375 0.03 0.0" rpy="0 0 ${pi/2}" />
+        <origin xyz="-0.105 0.035 0.0" rpy="0 0 ${pi/2}" />
     </joint>
-    <xacro:servo name="arm_servo_1"/>
+    <xacro:servo name="arm_servo_1" flipped="false"/>
     <joint name="plate_2_joint" type="fixed">
         <parent link="arm_servo_1_axis" />
         <child link="plate_2" />
-        <origin xyz="0.0425 0 0.0185" rpy="0 0 0" />
+        <origin xyz="0 -0.0425 0.0185" rpy="0 0 ${-pi/2}" />
     </joint>
     <joint name="plate_3_joint" type="fixed">
         <parent link="arm_servo_1_axis" />
         <child link="plate_3" />
-        <origin xyz="0.0425 0 -0.0185" rpy="0 0 0" />
+        <origin xyz="0 -0.0425 -0.0185" rpy="0 0 ${-pi/2}" />
     </joint>
     <xacro:plate plate_name="plate_2"/>
@@ -67,7 +70,7 @@
         <parent link="arm_servo_1_axis" />
         <child link="gripper_servo" />
-        <origin xyz="0.1 0.0 0.0" rpy="${-pi/2} 0 0" />
+        <origin xyz="0.0 -0.105 0.0" rpy="${-pi/2} 0 ${-pi/2}" />
     </joint>
-    <xacro:servo name="gripper_servo"/>
+    <xacro:servo name="gripper_servo" flipped="false"/>
     <joint name="gripper_gear_joint" type="fixed">
         <parent link="gripper_servo_axis" />

File: src/quac/description/urdf/servo.xacro (robot description, xacro)
@@ -4,5 +4,5 @@
     <xacro:property name="servo_y" value="0.025"/>
     <xacro:property name="servo_z" value="0.035"/>
-    <xacro:macro name="servo_macro" params="name">
+    <xacro:macro name="servo" params="name flipped">
         <link name="${name}">
             <visual>
@@ -28,5 +28,5 @@
                     <cylinder radius="0.002" length="0.08" />
                 </geometry>
-                <material name="red" />
+                <material name="yellow" />
             </visual>
             <xacro:inertial_cylinder mass="0.1" length="0.08" radius="0.002">
@@ -34,22 +34,15 @@
             </xacro:inertial_cylinder>
         </link>
-    </xacro:macro>
-    <xacro:macro name="servo" params="name">
-        <xacro:servo_macro name="${name}"/>
-        <joint name="${name}_joint" type="revolute">
-            <parent link="${name}" />
-            <child link="${name}_axis" />
-            <axis xyz="0 0 -1" />
-            <limit lower="-1.57" upper="1.57" effort="1" velocity="1" />
+        <joint name="${name}_joint" type="continuous">
+            <xacro:unless value="${flipped}">
+                <parent link="${name}" />
+                <child link="${name}_axis" />
+            </xacro:unless>
+            <xacro:if value="${flipped}">
+                <parent link="${name}_axis" />
+                <child link="${name}" />
+            </xacro:if>
+            <axis xyz="0 0 1" />
         </joint>
     </xacro:macro>
-    <xacro:macro name="servo_flipped" params="name">
-        <joint name="${name}_joint" type="revolute">
-            <parent link="${name}_axis" />
-            <child link="${name}" />
-            <axis xyz="0 0 -1" />
-            <limit lower="-1.57" upper="1.57" effort="1" velocity="1" />
-        </joint>
-        <xacro:servo_macro name="${name}"/>
-    </xacro:macro>
 </robot>

File: src/quac/worlds/obstacles.sdf.xacro (robot description, xacro)
@@ -1,4 +1,4 @@
 <sdf version='1.9' xmlns:xacro="http://www.ros.org/wiki/xacro">
-  <world name='empty'>
+  <world name='obstacles'>
     <physics name='1ßms' type='ignored'>
       <max_step_size>0.01</max_step_size>
@@ -12,4 +12,5 @@
       <render_engine>ogre2</render_engine>
     </plugin>
+    <plugin name='gz::sim::systems::Imu' filename='gz-sim-imu-system'></plugin>
     <plugin name='gz::sim::systems::Contact' filename='gz-sim-contact-system'/>
     <gravity>0 0 -9.8000000000000007</gravity>
