Commit message: yolo detection server

File: src/quac/description/gazebo.xacro (robot description, xacro)
@@ -58,4 +58,5 @@
                 <remapping>/robot_description:=robot_description</remapping>
                 <remapping>/tf:=tf</remapping>
+                <remapping>/tf_static:=tf_static</remapping>
                 <remapping>/clock:=clock</remapping>
                 <remapping>diff_drive_controller/cmd_vel_unstamped:=cmd_vel</remapping>

File: src/quac/description/robot.urdf.xacro (robot description, xacro)
@@ -4,4 +4,5 @@
     <xacro:include filename="urdf/inertial_macros.xacro" />
     <xacro:include filename="urdf/servo.xacro" />
+    <xacro:include filename="$(find realsense2_description)/urdf/_d435.urdf.xacro" />
     <xacro:include filename="urdf/chassis.xacro" />
     <xacro:include filename="urdf/wheels.xacro" />

File: src/quac/description/urdf/chassis.xacro (robot description, xacro)
@@ -44,9 +44,15 @@
     </joint>
     <link name="imu"/>
-    <joint name="camera_back_joint" type="fixed">
+    <!-- <joint name="camera_back_joint" type="fixed">
         <parent link="chassis"/>
         <child link="camera_back"/>
         <origin xyz="-0.09 0.0 0.1" rpy="0 0 ${pi}"/>
     </joint>
-    <link name="camera_back"/>
+    <link name="camera_back"/> -->
+    <xacro:arg name="use_nominal_extrinsics" default="false"/>
+    <xacro:arg name="add_plug" default="true" />
+    <xacro:arg name="use_mesh" default="true" />
+    <xacro:sensor_d435 parent="chassis" name="camera_back" use_nominal_extrinsics="$(arg use_nominal_extrinsics)" add_plug="$(arg add_plug)" use_mesh="$(arg use_mesh)">
+        <origin xyz="-0.09 0.0 0.1" rpy="0 0 ${pi}"/>
+    </xacro:sensor_d435>
 </robot>

Commit message: fixes + realsense urdf

File: src/quac/description/gazebo.xacro (robot description, xacro)
@@ -92,5 +92,5 @@
     </gazebo>
     <xacro:macro name="cam_sim" params="frame">
-        <gazebo reference="${frame}_depth_optical_frame">
+        <gazebo reference="${frame}_depth_frame">
             <sensor name="${frame}_sim" type="rgbd_camera">
                 <always_on>true</always_on>
@@ -98,5 +98,5 @@
                 <update_rate>10</update_rate>
                 <topic>${frame}</topic>
-                <gz_frame_id>${frame}_depth_optical_frame</gz_frame_id>
+                <gz_frame_id>${frame}_depth_frame</gz_frame_id>
                 <camera>
                 <horizontal_fov>1.48702</horizontal_fov>

File: src/quac/description/robot.urdf.xacro (robot description, xacro)
@@ -4,5 +4,5 @@
     <xacro:include filename="urdf/inertial_macros.xacro" />
     <xacro:include filename="urdf/servo.xacro" />
-    <xacro:include filename="$(find realsense2_description)/urdf/_d435.urdf.xacro" />
+    <xacro:include filename="urdf/d435.xacro" />
     <xacro:include filename="urdf/chassis.xacro" />
     <xacro:include filename="urdf/wheels.xacro" />

File: src/quac/description/urdf/arm.xacro (robot description, xacro)
@@ -94,5 +94,5 @@
         </xacro:inertial_cylinder>
     </link>
-    <xacro:sensor_d435 parent="gripper_servo" name="camera_front" use_nominal_extrinsics="true" add_plug="false" use_mesh="true">
+    <xacro:sensor_d435 parent="gripper_servo" name="camera_front" use_nominal_extrinsics="true">
         <origin xyz="0 0 0" rpy="0 0 0"/>
     </xacro:sensor_d435>

File: src/quac/description/urdf/chassis.xacro (robot description, xacro)
@@ -26,10 +26,4 @@
         </visual>
     </link>
-    <gazebo reference="chassis">
-        <material>Gazebo/White</material>
-        <mu1>0.2</mu1>
-        <mu2>0.2</mu2>
-        <gravity>true</gravity>
-    </gazebo>
     <joint name="laser_joint" type="fixed">
         <parent link="chassis"/>
@@ -44,6 +38,6 @@
     </joint>
     <link name="imu"/>
-    <xacro:sensor_d435 parent="chassis" name="camera_back" use_nominal_extrinsics="true" add_plug="false" use_mesh="true">
-        <origin xyz="-0.09 0.0 0.1" rpy="0 0 ${pi}"/>
+    <xacro:sensor_d435 parent="chassis" name="camera_back" use_nominal_extrinsics="true">
+        <origin xyz="-0.1 0.0 0.09" rpy="0 0 ${pi}"/>
     </xacro:sensor_d435>
 </robot>

File: src/quac/description/urdf/wheels.xacro (robot description, xacro)
@@ -34,7 +34,4 @@
             </xacro:inertial_cylinder>
         </link>
-        <gazebo reference="${name}">
-            <material>Gazebo/Black</material>
-        </gazebo>
     </xacro:macro>
     <!-- Four wheels -->

Commit message: inertias

File: src/quac/description/gazebo.xacro (robot description, xacro)
@@ -127,5 +127,5 @@
         </gazebo>
     </xacro:macro>
-    <xacro:cam_sim frame="camera_front"/>
+    <xacro:cam_sim frame="camera_gripper"/>
     <xacro:cam_sim frame="camera_back"/>
     <gazebo reference="imu">

File: src/quac/description/urdf/version_6/arm.xacro (robot description, xacro)
@@ -14,4 +14,9 @@
     </joint>
     <link name="arm_segment_1">
+        <inertial>
+            <origin xyz="0 0 0" rpy="0 0 0"/>
+            <mass value="0.2"/>
+            <inertia ixx="0.01" ixy="0.0" ixz="0.0" iyy="0.01" iyz="0.0" izz="0.01"/>
+        </inertial>
         <visual>
             <origin xyz="0 0 0" rpy="${-pi/2} 0 0"/>
@@ -29,4 +34,9 @@
     </joint>
     <link name="arm_segment_2">
+        <inertial>
+            <origin xyz="0 0 0" rpy="0 0 0"/>
+            <mass value="0.2"/>
+            <inertia ixx="0.01" ixy="0.0" ixz="0.0" iyy="0.01" iyz="0.0" izz="0.01"/>
+        </inertial>
         <visual>
             <origin xyz="0 0 0" rpy="${-pi/2} 0 0"/>
@@ -46,5 +56,11 @@
         <axis xyz="0 0 1" />
     </joint>
-    <link name="gripper_gear"></link>
+    <link name="gripper_gear">
+        <inertial>
+            <origin xyz="0 0 0" rpy="0 0 0"/>
+            <mass value="0.1"/>
+            <inertia ixx="0.01" ixy="0.0" ixz="0.0" iyy="0.01" iyz="0.0" izz="0.01"/>
+        </inertial>
+    </link>
     <xacro:macro name="gripper_side" params="side multiplier">
         <joint name="gripper_${side}_back_piece_joint" type="continuous">
@@ -56,4 +72,9 @@
         </joint>
         <link name="gripper_${side}_back_piece">
+            <inertial>
+                <origin xyz="0 0 0" rpy="0 0 0"/>
+                <mass value="0.02"/>
+                <inertia ixx="0.01" ixy="0.0" ixz="0.0" iyy="0.01" iyz="0.0" izz="0.01"/>
+            </inertial>
             <visual>
                 <origin xyz="0 0 0" rpy="0 0 ${pi/2+multiplier*pi/2}"/>
@@ -72,4 +93,9 @@
         </joint>
         <link name="gripper_${side}_front_piece">
+            <inertial>
+                <origin xyz="0 0 0" rpy="0 0 0"/>
+                <mass value="0.02"/>
+                <inertia ixx="0.01" ixy="0.0" ixz="0.0" iyy="0.01" iyz="0.0" izz="0.01"/>
+            </inertial>
             <visual>
                 <origin xyz="0 0 0" rpy="0 0 ${pi/2+multiplier*pi/2}"/>
@@ -88,4 +114,9 @@
         </joint>
         <link name="gripper_${side}">
+            <inertial>
+                <origin xyz="0 0 0" rpy="0 0 0"/>
+                <mass value="0.1"/>
+                <inertia ixx="0.01" ixy="0.0" ixz="0.0" iyy="0.01" iyz="0.0" izz="0.01"/>
+            </inertial>
             <visual>
                 <origin xyz="0 0 0" rpy="0 0 0"/>

Commit message: new arm

File: src/quac/description/gazebo.xacro (robot description, xacro)
@@ -30,24 +30,21 @@
             <plugin>gz_ros2_control/GazeboSimSystem</plugin>
         </hardware>
-        <joint name="arm_servo_0_joint">
+        <joint name="arm_segment_0_joint">
             <command_interface name="position"/>
             <command_interface name="velocity"/>
             <state_interface name="position"/>
             <state_interface name="velocity"/>
-            <state_interface name="torque"/>
         </joint>
-        <joint name="arm_servo_1_joint">
+        <joint name="arm_segment_1_joint">
             <command_interface name="position"/>
             <command_interface name="velocity"/>
             <state_interface name="position"/>
             <state_interface name="velocity"/>
-            <state_interface name="torque"/>
         </joint>
-        <joint name="gripper_servo_joint">
+        <joint name="gripperjoint">
             <command_interface name="position"/>
             <command_interface name="velocity"/>
             <state_interface name="position"/>
             <state_interface name="velocity"/>
-            <state_interface name="torque"/>
         </joint>
     </ros2_control>

File: src/quac/description/ros2_control.xacro (robot description, xacro)
@@ -4,4 +4,5 @@
     <xacro:arg name="disable_wheels" default="false"/>
     <xacro:arg name="disable_arm" default="false"/>
+    <xacro:arg name="old_arm" default="false"/>
     <!-- WHEELS -->
     <ros2_control name="wheel_hardware" type="system">
@@ -64,7 +65,14 @@
             </joint>
         </xacro:macro>
-        <xacro:arm_joint name="arm_servo_0_joint"   id="5" inverted="true" offset="${pi/2}" pos_min="${-pi}" pos_max="0"/>
-        <xacro:arm_joint name="arm_servo_1_joint"   id="6" inverted="false"  offset="${1.8-pi/2}"   pos_min="0"     pos_max="${pi/2 + 0.8}"/>
-        <xacro:arm_joint name="gripper_servo_joint" id="1" inverted="true"  offset="1.75"  pos_min="0"        pos_max="1.7" />
+        <xacro:arm_joint name="gripper_joint" id="1" inverted="true"  offset="1.75"        pos_min="0"      pos_max="1.7" />
+        <xacro:if value="$(arg old_arm)">
+            <xacro:arm_joint name="arm_segment_0_joint"   id="5" inverted="true"  offset="${pi/2}"     pos_min="${-pi}" pos_max="0"/>
+            <xacro:arm_joint name="arm_segment_1_joint"   id="6" inverted="false" offset="${1.8-pi/2}" pos_min="0"      pos_max="${pi/2 + 0.8}"/>
+        </xacro:if>
+        <xacro:unless value="$(arg old_arm)">
+            <xacro:arm_joint name="arm_segment_0_joint"   id="" inverted=""  offset=""     pos_min="" pos_max=""/>
+            <xacro:arm_joint name="arm_segment_1_joint"   id="" inverted="" offset="" pos_min=""      pos_max=""/>
+            <xacro:arm_joint name="arm_segment_2_joint"   id="" inverted=""  offset=""        pos_min=""      pos_max="" />
+        </xacro:unless>
     </ros2_control>
 </robot>

File: src/quac/description/urdf/version_6/chassis.xacro (robot description, xacro)
@@ -1,5 +1,10 @@
 <?xml version="1.0"?>
 <robot xmlns:xacro="http://www.ros.org/wiki/xacro">
-    <xacro:include filename="arm.xacro" />
+    <xacro:unless value="$(arg old_arm)">
+        <xacro:include filename="arm_v2.xacro" />
+    </xacro:unless>
+    <xacro:if value="$(arg old_arm)">
+        <xacro:include filename="arm_v1.xacro" />
+    </xacro:if>
     <xacro:include filename="wheels.xacro" />
     <material name="chassis_material">

File: src/quac/description/urdf/version_6/gripper.xacro (robot description, xacro)
@@ -1,60 +1,24 @@
 <?xml version="1.0"?>
 <robot xmlns:xacro="http://www.ros.org/wiki/xacro">
-<material name="gripper_material">
-    <color rgba="0.7 0.2 0.2 1.0" />
-</material>
-<material name="arm_material">
-    <color rgba="0.7 0.7 0.7 1.0" />
-</material>
-    <joint name="arm_servo_0_joint" type="continuous">
-        <parent link="chassis"/>
-        <child link="arm_segment_1"/>
-        <origin xyz="0.13 0 0.04475" rpy="${pi/2} 0 0"/>
+    <material name="gripper_material">
+        <color rgba="0.7 0.2 0.2 1.0" />
+    </material>
+    <link name="gripper_base">
+        <inertial>
+            <origin xyz="0 0 0" rpy="0 0 0"/>
+            <mass value="0.1"/>
+            <inertia ixx="0.01" ixy="0.0" ixz="0.0" iyy="0.01" iyz="0.0" izz="0.01"/>
+        </inertial>
+    </link>
+    <xacro:sensor_d435 parent="gripper_base" name="camera_gripper" use_nominal_extrinsics="true">
+        <origin xyz="0.022 -0.0255 0.0225" rpy="0 0 0"/>
+    </xacro:sensor_d435>
+    <joint name="gripper_joint" type="continuous">
+        <parent link="gripper_base" />
+        <child link="gripper_link" />
+        <origin xyz="-0.0207 0.0125 0.0355" rpy="0 0 0"/>
         <axis xyz="0 0 1" />
     </joint>
-    <link name="arm_segment_1">
-        <inertial>
-            <origin xyz="0 0 0" rpy="0 0 0"/>
-            <mass value="0.2"/>
-            <inertia ixx="0.01" ixy="0.0" ixz="0.0" iyy="0.01" iyz="0.0" izz="0.01"/>
-        </inertial>
-        <visual>
-            <origin xyz="0 0 0" rpy="${-pi/2} 0 0"/>
-            <geometry>
-                <mesh filename="package://quac/meshes/version_6/arm_segment_1_reduced.stl" scale="${mesh_scale} ${mesh_scale} ${mesh_scale}"/>
-            </geometry>
-            <material name="arm_material"/>
-        </visual>
-    </link>
-    <joint name="arm_servo_1_joint" type="continuous">
-        <parent link="arm_segment_1"/>
-        <child link="arm_segment_2"/>
-        <origin xyz="-0.1025 0.0287 0" rpy="0 0 0"/>
-        <axis xyz="0 0 1" />
-    </joint>
-    <link name="arm_segment_2">
-        <inertial>
-            <origin xyz="0 0 0" rpy="0 0 0"/>
-            <mass value="0.2"/>
-            <inertia ixx="0.01" ixy="0.0" ixz="0.0" iyy="0.01" iyz="0.0" izz="0.01"/>
-        </inertial>
-        <visual>
-            <origin xyz="0 0 0" rpy="${-pi/2} 0 0"/>
-            <geometry>
-                <mesh filename="package://quac/meshes/version_6/arm_segment_2_reduced.stl" scale="${mesh_scale} ${mesh_scale} ${mesh_scale}"/>
-            </geometry>
-            <material name="arm_material"/>
-        </visual>
-    </link>
-    <xacro:sensor_d435 parent="arm_segment_2" name="camera_gripper" use_nominal_extrinsics="true">
-        <origin xyz="0.09 0.025 0.025" rpy="${-pi/2} 0 0"/>
-    </xacro:sensor_d435>
-    <joint name="gripper_servo_joint" type="continuous">
-        <parent link="arm_segment_2" />
-        <child link="gripper_gear" />
-        <origin xyz="0.0483 0.04 -0.0125" rpy="${-pi/2} 0 0"/>
-        <axis xyz="0 0 1" />
-    </joint>
-    <link name="gripper_gear">
+    <link name="gripper_link">
         <inertial>
             <origin xyz="0 0 0" rpy="0 0 0"/>
@@ -65,8 +29,8 @@
     <xacro:macro name="gripper_side" params="side multiplier">
         <joint name="gripper_${side}_back_piece_joint" type="continuous">
-            <parent link="arm_segment_2" />
+            <parent link="gripper_base" />
             <child link="gripper_${side}_back_piece" />
-            <origin xyz="0.048 0.015 ${multiplier * 0.0315}" rpy="${-pi/2} 0 0"/>
-            <mimic joint="gripper_servo_joint" multiplier="${-multiplier}" offset="${multiplier * pi/2}"/>
+            <origin xyz="-0.021 ${-multiplier * 0.0315} 0.0105" rpy="0 0 0"/>
+            <mimic joint="gripper_joint" multiplier="${-multiplier}" offset="${multiplier * pi/2}"/>
             <axis xyz="0 0 1" />
         </joint>
@@ -86,8 +50,8 @@
         </link>
         <joint name="gripper_${side}_front_piece_joint" type="continuous">
-            <parent link="arm_segment_2" />
+            <parent link="gripper_base" />
             <child link="gripper_${side}_front_piece" />
-            <origin xyz="0.069 0.0045 ${multiplier * 0.0105}" rpy="${-pi/2} 0 0"/>
-            <mimic joint="gripper_servo_joint" multiplier="${-multiplier}" offset="${multiplier * pi/2}"/>
+            <origin xyz="0.0 ${-multiplier * 0.0105} 0.0" rpy="0 0 0"/>
+            <mimic joint="gripper_joint" multiplier="${-multiplier}" offset="${multiplier * pi/2}"/>
             <axis xyz="0 0 1" />
         </joint>
@@ -110,5 +74,5 @@
             <child link="gripper_${side}" />
             <origin xyz="0.0 ${-multiplier * 0.043} 0.006" rpy="0 0 0"/>
-            <mimic joint="gripper_servo_joint" multiplier="${multiplier}" offset="${-multiplier * pi/2}"/>
+            <mimic joint="gripper_joint" multiplier="${multiplier}" offset="${-multiplier * pi/2}"/>
             <axis xyz="0 0 1" />
         </joint>
