Commit message: docker setup, bugfixes, params, launch

File: src/quac/description/ros2_control.xacro (robot description, xacro)
@@ -85,9 +85,9 @@
                 <remapping>/tf:=tf</remapping>
                 <remapping>/clock:=clock</remapping>
-                <remapping>diff_drive_controller/cmd_vel:=cmd_vel</remapping>
+                <remapping>diff_drive_controller/cmd_vel_unstamped:=cmd_vel</remapping>
                 <remapping>diff_drive_controller/odom:=odom</remapping>
                 <remapping>arm_position_controller/joint_trajectory:=arm_joint_trajectory</remapping>
             </ros>
-            <parameters>$(find quac)/config/controllers.yaml</parameters>
+            <parameters>$(find quac)/config/control.yaml</parameters>
             <parameters>$(find quac)/config/gz_sim_time.yaml</parameters>
         </plugin>

File: src/quac/description/urdf/arm.xacro (robot description, xacro)
@@ -31,5 +31,5 @@
         <parent link="chassis" />
         <child link="arm_servo_0_axis" />
-        <origin xyz="0.135 0.0 0.04" rpy="${pi/2} ${pi/2} 0" />
+        <origin xyz="0.135 0.0 0.064" rpy="${pi/2} ${pi/2} 0" />
     </joint>
     <xacro:servo_flipped name="arm_servo_0"/>

File: src/quac/description/urdf/chassis.xacro (robot description, xacro)
@@ -25,10 +25,4 @@
             <material name="chassis_material"/>
         </visual>
-        <collision>
-            <origin xyz="0 0 0" rpy="0 0 0"/>
-            <geometry>
-                <mesh filename="package://quac/meshes/chassis.stl" scale="${mesh_scale} ${mesh_scale} ${mesh_scale}"/>
-            </geometry>
-        </collision>
     </link>
     <gazebo reference="chassis">

File: src/quac/worlds/obstacles.sdf.xacro (robot description, xacro)
@@ -1,3 +1,3 @@
-<sdf version='1.10' xmlns:xacro="http://www.ros.org/wiki/xacro">
+<sdf version='1.9' xmlns:xacro="http://www.ros.org/wiki/xacro">
   <world name='empty'>
     <physics name='1ßms' type='ignored'>

Commit message: config

File: src/quac/description/ros2_control.xacro (robot description, xacro)
@@ -9,5 +9,5 @@
             <xacro:unless value="$(arg disable_wheels)">
                 <plugin>quac_hardware/DDSM115</plugin>
-                <param name="port">/dev/ttyTCU0</param>
+                <param name="port">/dev/quac/ddsm115</param>
                 <param name="act">3</param>
             </xacro:unless>
@@ -26,8 +26,8 @@
             </joint>
         </xacro:macro>
-        <xacro:wheel_joint name="wheel_front_left_joint" id="4" scalar="1"/>
-        <xacro:wheel_joint name="wheel_front_right_joint" id="1" scalar="-1"/>
+        <xacro:wheel_joint name="wheel_front_left_joint" id="1" scalar="1"/>
+        <xacro:wheel_joint name="wheel_front_right_joint" id="2" scalar="-1"/>
         <xacro:wheel_joint name="wheel_rear_left_joint" id="3" scalar="1"/>
-        <xacro:wheel_joint name="wheel_rear_right_joint" id="2" scalar="-1"/>
+        <xacro:wheel_joint name="wheel_rear_right_joint" id="4" scalar="-1"/>
     </ros2_control>
     <!-- ARM -->
@@ -36,5 +36,5 @@
             <xacro:unless value="$(arg disable_arm)">
                 <plugin>quac_hardware/WaveshareServos</plugin>
-                <param name="port">/dev/quac/arm_servos</param>
+                <param name="port">/dev/quac/servos</param>
                 <param name="crawler_arm_param_hw_start_duration_sec">0</param>
                 <param name="crawler_arm_hw_stop_duration_sec">3.0</param>

File: src/quac/description/urdf/chassis.xacro (robot description, xacro)
@@ -29,5 +29,5 @@
         <parent link="chassis"/>
         <child link="laser"/>
-        <origin xyz="-0.02 0.0 0.15" rpy="0 0 ${pi}"/>
+        <origin xyz="-0.02 0.0 0.15" rpy="0 0 ${pi/2}"/>
     </joint>
     <link name="laser"/>

Commit message: rtabmap + a bunch of other things

File: src/quac/description/ros2_control.xacro (robot description, xacro)
@@ -14,4 +14,5 @@
             <xacro:if value="$(arg disable_wheels)">
                 <plugin>mock_components/GenericSystem</plugin>
+                <param name="calculate_dynamics">true</param>
             </xacro:if>
         </hardware>

File: src/quac/description/urdf/oak_d_lite.xacro (robot description, xacro)
@@ -4,15 +4,14 @@
         <color rgba="0.5 0.5 0.5 1"/>
     </material>
-	<xacro:macro name="base"
-		params="camera_name parent has_imu cam_pos_x cam_pos_y cam_pos_z cam_roll cam_pitch cam_yaw">
-		<!-- base_link of the sensor-->
+	<xacro:macro name="oak_d_lite" params="camera_name parent xyz rpy">
+		<xacro:property name="baseline" value="0.075" />
+		<xacro:property name="left_name" value="infra2" />
+		<xacro:property name="right_name" value="infra1" />
 		<link name="${camera_name}" />
 		<joint name="${camera_name}_center_joint" type="fixed">
 			<parent link="${parent}" />
 			<child link="${camera_name}" />
-			<origin xyz="${cam_pos_x} ${cam_pos_y} ${cam_pos_z}"
-				rpy="${cam_roll} ${cam_pitch} ${cam_yaw}" />
+			<origin xyz="${xyz}" rpy="${rpy}" />
 		</joint>
-		<!-- device Center -->
 		<link name="${camera_name}_model_origin">
 			<visual>
@@ -27,28 +26,6 @@
 			<parent link="${camera_name}" />
 			<child link="${camera_name}_model_origin" />
-			<origin xyz="0 0 0" rpy="1.5708 0 1.5708" />
+			<origin xyz="0 0 0" rpy="${pi/2} 0 ${pi/2}" />
 		</joint>
-		<!-- IMU -->
-		<xacro:if value="${has_imu}">
-			<link name="${camera_name}_imu_frame" />
-			<joint name="${camera_name}_imu_joint" type="fixed">
-				<parent link="${camera_name}" />
-				<child link="${camera_name}_imu_frame" />
-				<origin xyz="${imu_offset_x} ${imu_offset_y} ${imu_offset_z}"
-					rpy="${imu_r} ${imu_p} ${imu_y}" />
-			</joint>
-		</xacro:if>
-	</xacro:macro>
-	<xacro:macro name="oak_d_lite"
-		params="camera_name parent
-                                           cam_pos_x cam_pos_y cam_pos_z
-                                           cam_roll cam_pitch cam_yaw">
-		<xacro:property name="has_imu" value="false" />
-		<xacro:property name="baseline" value="0.075" />
-		<xacro:property name="left_name" value="infra2" />
-		<xacro:property name="right_name" value="infra1" />
-		<xacro:base camera_name="${camera_name}" parent="${parent}" has_imu="${has_imu}"
-			cam_pos_x="${cam_pos_x}" cam_pos_y="${cam_pos_y}" cam_pos_z="${cam_pos_z}"
-			cam_roll="${cam_roll}" cam_pitch="${cam_pitch}" cam_yaw="${cam_yaw}" />
 		<!-- RGB Camera -->
 		<link name="${camera_name}_color_frame" />
@@ -57,4 +34,10 @@
 			<child link="${camera_name}_color_frame" />
 			<origin xyz="0 0 0" rpy="0 0 0" />
+		</joint>
+		<link name="${camera_name}_imu"/>
+		<joint name="${camera_name}_imu_joint" type="fixed">
+			<parent link="${camera_name}_color_frame"/>
+			<child link="${camera_name}_imu"/>
+			<origin xyz="-0.00315 0.0006439 -0.0002" rpy="-${pi/2} 0.0 ${pi/2}"/>
 		</joint>
 		<link name="${camera_name}_color_optical_frame" />

File: src/quac/description/urdf/version_6/chassis.xacro (robot description, xacro)
@@ -9,5 +9,5 @@
         <parent link="base_link"/>
         <child link="chassis"/>
-        <origin xyz="0 0 0.125" rpy="0 0 0"/>
+        <origin xyz="0 0 0.13" rpy="0 0 0"/>
     </joint>
     <link name="chassis">
@@ -31,13 +31,7 @@
     </joint>
     <link name="laser"/>
-    <joint name="imu_joint" type="fixed">
-        <parent link="chassis"/>
-        <child link="imu"/>
-        <origin xyz="0.15 0 0.01" rpy="0 0 ${-pi/2}"/>
-    </joint>
-    <link name="imu"/>
     <xacro:sensor_d435 parent="chassis" name="camera_back" use_nominal_extrinsics="true">
         <origin xyz="-0.09 0.0 0.09" rpy="0 0 ${pi}"/>
     </xacro:sensor_d435>
-	<xacro:oak_d_lite camera_name="camera_front" parent="chassis" cam_pos_x="0.16" cam_pos_y="0" cam_pos_z="-0.015" cam_roll="0" cam_pitch="0" cam_yaw="0"/>
+	<xacro:oak_d_lite camera_name="camera_front" parent="chassis" xyz="0.16 0 -0.025" rpy="${pi} 0 0"/>
 </robot>

Commit message: arm config

File: src/quac/description/ros2_control.xacro (robot description, xacro)
@@ -71,7 +71,7 @@
         </xacro:if>
         <xacro:unless value="$(arg old_arm)">
-            <xacro:arm_joint name="arm_segment_0_joint"   id="1" inverted="false"  offset="${3*pi/2}"     pos_min="${-pi-pi/8}"   pos_max="0"/>
-            <xacro:arm_joint name="arm_segment_1_joint"   id="2" inverted="false"  offset="${pi/2}"   pos_min="0"        pos_max="${pi}"/>
-            <xacro:arm_joint name="arm_segment_2_joint"   id="3" inverted="true"   offset="${pi}" pos_min="${-pi/5}" pos_max="${pi/2}" />
+            <xacro:arm_joint name="arm_segment_0_joint"   id="1" inverted="false"  offset="${3*pi/2}"     pos_min="${-5*pi/4 - 0.1}"   pos_max="0"/>
+            <xacro:arm_joint name="arm_segment_1_joint"   id="2" inverted="false"  offset="${pi}"   pos_min="${-pi/4}"        pos_max="${pi/2}"/>
+            <xacro:arm_joint name="arm_segment_2_joint"   id="3" inverted="true"   offset="${3*pi/2}" pos_min="0" pos_max="${pi - 0.05}" />
         </xacro:unless>
     </ros2_control>

File: src/quac/description/urdf/version_6/arm_v2.xacro (robot description, xacro)
@@ -8,5 +8,5 @@
         <parent link="chassis"/>
         <child link="arm_segment_0"/>
-        <origin xyz="0.13 0 0.0445" rpy="${pi/2} 0 0"/>
+        <origin xyz="0.15 0 0.0445" rpy="${pi/2} 0 0"/>
         <axis xyz="0 0 1" />
     </joint>
@@ -38,5 +38,5 @@
         </inertial>
         <visual>
-            <origin xyz="0 0 0" rpy="${-pi/2} 0 0"/>
+            <origin xyz="-0.02 0.05 0" rpy="${pi/2} 0 0"/>
             <geometry>
                 <mesh filename="package://quac/meshes/version_6/arm_v2/arm_segment_1_reduced.stl" scale="${mesh_scale} ${mesh_scale} ${mesh_scale}"/>
@@ -48,5 +48,5 @@
         <parent link="arm_segment_1"/>
         <child link="arm_segment_2"/>
-        <origin xyz="0.02 0.05 0" rpy="0 0 0"/>
+        <origin xyz="-0.02 0.05 0" rpy="0 0 0"/>
         <axis xyz="0 0 1" />
     </joint>
