Commit message: ekf

File: src/quac/description/urdf/version_6/chassis.xacro (robot description, xacro)
@@ -40,5 +40,5 @@
         <parent link="chassis"/>
         <child link="imu"/>
-        <origin xyz="-0.035 -0.06 0.095" rpy="0 0 0"/>
+        <origin xyz="0.15 0 0.01" rpy="0 0 ${-pi/2}"/>
     </joint>
     <link name="imu"/>

Commit message: param adjustments

File: src/quac/description/urdf/version_6/chassis.xacro (robot description, xacro)
@@ -28,5 +28,5 @@
         <parent link="chassis"/>
         <child link="laser"/>
-        <origin xyz="-0.035 0.0 0.127" rpy="0 0 ${pi/2}"/>
+        <origin xyz="-0.035 0.0 0.127" rpy="0 0 ${-pi/2}"/>
     </joint>
     <link name="laser"/>
